Commit message: Modified robot model parameters

File: urdf/manipulator.urdf (robot description, URDF)
Before this commit: robot manipulator, 9 links, 8 joints
Links:
- link intermediate_link: mass 0.95 -> 0.18
- link padding_link: mass 0.01 -> 0.005
- link proximal_link: mass 1.0 -> 0.18
- link tip_link: mass 0.2 -> 0.02
Joints:
- joint holder_to_proximal: limit lower=-1.5708 upper=1.5708 effort=1000 velocity=1000 -> lower=0 upper=3.14159265359 effort=1000 velocity=1000; origin xyz=0 0 0 -> xyz=0 0 0 rpy=0 -1.5708 0
- joint intermediate_to_tip: limit lower=-3.00197 upper=3.00197 effort=1000 velocity=1000 -> lower=0 upper=6.00394 effort=1000 velocity=1000; origin xyz=0 -0.16 0 -> xyz=0 -0.16 0 rpy=-3.00197 0 0
- joint proximal_to_intermediate: limit lower=-2.9234265 upper=2.9234265 effort=1000 velocity=1000 -> lower=-5.846853 upper=0 effort=1000 velocity=1000; origin xyz=0.014 0.02695 0 -> xyz=0.014 0.02695 0 rpy=2.9234265 0 0

File: xacro/manipulator.urdf.xacro (robot description, xacro)
@@ -22,15 +22,15 @@
     <xacro:property name="proximal_y" value="0.2115"/>
     <xacro:property name="proximal_z" value="0.047138" />
-    <xacro:property name="proximal_m" value="1.0" />
+    <xacro:property name="proximal_m" value="0.180" />
     <!-- Intermediate link Inertia -->
     <xacro:property name="intermediate_x" value="0.0419"/>
     <xacro:property name="intermediate_y" value="0.206"/>
     <xacro:property name="intermediate_z" value="0.044276" />
-    <xacro:property name="intermediate_m" value="0.95" />
+    <xacro:property name="intermediate_m" value="0.180" />
     <!-- Tip link Inertia -->
     <xacro:property name="tip_x" value="0.027317"/>
     <xacro:property name="tip_y" value="0.183"/>
     <xacro:property name="tip_z" value="0.024" />
-    <xacro:property name="tip_m" value="0.2" />
+    <xacro:property name="tip_m" value="0.02" />
     <mujoco>
         <compiler meshdir="../meshes/${mesh_ext}/" balanceinertia="true" discardvisual="false" />
@@ -116,7 +116,7 @@
         <parent link="holder_link"/>
         <child link="proximal_link"/>
-        <limit effort="1000" lower="-1.5708" upper="1.5708" velocity="1000"/>
+        <limit effort="1000" lower="0" upper="3.14159265359" velocity="1000"/>
         <axis rpy="0 0 0" xyz="0 1 0"/>
-        <origin xyz="0 0 0"/>
+        <origin rpy="0 -1.5708 0" xyz="0 0 0"/>
     </joint>
     <xacro:my_link
@@ -152,7 +152,7 @@
         <parent link="proximal_link"/>
         <child link="intermediate_link"/>
-        <limit effort="1000" lower="-2.9234265" upper="2.9234265" velocity="1000"/>
+        <limit effort="1000" lower="-5.846853" upper="0" velocity="1000"/>
         <axis rpy="0 0 0" xyz="1 0 0"/>
-        <origin xyz="0.014 0.02695 0"/>
+        <origin rpy="2.9234265 0 0" xyz="0.014 0.02695 0"/>
     </joint>
     <xacro:my_link
@@ -171,7 +171,7 @@
         <parent link="intermediate_link"/>
         <child link="tip_link"/>
-        <limit effort="1000" lower="-3.00197" upper="3.00197" velocity="1000"/>
+        <limit effort="1000" lower="0" upper="6.00394" velocity="1000"/>
         <axis rpy="0 0 0" xyz="1 0 0"/>
-        <origin xyz="0 -0.16 0"/>
+        <origin rpy="-3.00197 0 0" xyz="0 -0.16 0"/>
     </joint>
     <xacro:my_link
@@ -203,5 +203,5 @@
             y="0.01"
             z="0.01"
-            m="0.01"/>
+            m="0.005"/>
 <!--    <actuator>
         <motor name="holder_to_proximal"        gear="100" joint="holder_to_proximal" />
