Commit message: fixed direction of first degree of freedom and adjusted zero position

File: xacro/manipulator.urdf.xacro (robot description, xacro)
@@ -153,5 +153,5 @@
         <child link="intermediate_link"/>
         <limit effort="1000" lower="-5.846853" upper="0" velocity="1000"/>
-        <axis rpy="0 0 0" xyz="1 0 0"/>
+        <axis rpy="0 0 0" xyz="-1 0 0"/>
         <origin rpy="2.9234265 0 0" xyz="0.014 0.02695 0"/>
     </joint>
@@ -173,5 +173,5 @@
         <limit effort="1000" lower="0" upper="6.00394" velocity="1000"/>
         <axis rpy="0 0 0" xyz="1 0 0"/>
-        <origin rpy="-3.00197 0 0" xyz="0 -0.16 0"/>
+        <origin rpy="-2.9 0 0" xyz="0 -0.16 0"/>
     </joint>
     <xacro:my_link

Commit message: cleaned up xacro a bit

File: xacro/manipulator.urdf.xacro (robot description, xacro)
@@ -71,17 +71,4 @@
     <!-- World Link -->
     <link name="world"/>
-    <!-- Dummy Link -->
-    <link name="link0"/>
-    <joint name="world_joint" type="fixed">
-        <parent link="world"/>
-        <child link="link0"/>
-        <origin xyz="0 0 0" rpy="0 0 0"/>
-        <axis xyz="0 0 1"/>
-    </joint>
-    <joint name="holder_joint" type="fixed">
-        <parent link="link0"/>
-        <child link="holder_link"/>
-        <origin xyz="0 0 0" rpy="0 0 0"/>
-    </joint>
     <xacro:my_link
             name="holder_link"
@@ -96,9 +83,4 @@
             z="0.1"
             m="0.1"/>
-    <joint name="holder_to_stage" type="fixed">
-        <parent link="holder_link"/>
-        <child link="stage_link"/>
-        <origin xyz="0 0 -0.2665"/>
-    </joint>
     <xacro:my_link
             name="stage_link"
@@ -113,11 +95,4 @@
             z="0.1"
             m="5"/>
-    <joint name="holder_to_proximal" type="revolute">
-        <parent link="holder_link"/>
-        <child link="proximal_link"/>
-        <limit effort="1000" lower="0" upper="3.14159265359" velocity="1000"/>
-        <axis rpy="0 0 0" xyz="0 1 0"/>
-        <origin rpy="0 -1.5708 0" xyz="0 0 0"/>
-    </joint>
     <xacro:my_link
             name="proximal_link"
@@ -132,9 +107,16 @@
             z="${proximal_z}"
             m="${proximal_m}"/>
-    <joint name="holder_to_base" type="fixed">
-        <parent link="holder_link"/>
-        <child link="base_link"/>
-        <origin xyz="0 0.20595 0"/>
-    </joint>
+    <xacro:my_link
+            name="intermediate_link"
+            origin_rpy="0 0 0"
+            origin_xyz="0 0 0"
+            mesh_file="${intermediate_link_mesh}"
+            color_name="${color_name}"
+            color="${color}"
+            opacity="${opacity}"
+            x="${intermediate_x}"
+            y="${intermediate_y}"
+            z="${intermediate_z}"
+            m="${intermediate_m}"/>
     <xacro:my_link
             name="base_link"
@@ -149,30 +131,4 @@
             z="0.1"
             m="0.1"/>
-    <joint name="proximal_to_intermediate" type="revolute">
-        <parent link="proximal_link"/>
-        <child link="intermediate_link"/>
-        <limit effort="1000" lower="-5.846853" upper="0" velocity="1000"/>
-        <axis rpy="0 0 0" xyz="-1 0 0"/>
-        <origin rpy="2.9234265 0 0" xyz="0.014 0.02695 0"/>
-    </joint>
-    <xacro:my_link
-            name="intermediate_link"
-            origin_rpy="0 0 0"
-            origin_xyz="0 0 0"
-            mesh_file="${intermediate_link_mesh}"
-            color_name="${color_name}"
-            color="${color}"
-            opacity="${opacity}"
-            x="${intermediate_x}"
-            y="${intermediate_y}"
-            z="${intermediate_z}"
-            m="${intermediate_m}"/>
-    <joint name="intermediate_to_tip" type="revolute">
-        <parent link="intermediate_link"/>
-        <child link="tip_link"/>
-        <limit effort="1000" lower="0" upper="6.00394" velocity="1000"/>
-        <axis rpy="0 0 0" xyz="1 0 0"/>
-        <origin rpy="-2.9 0 0" xyz="0 -0.16 0"/>
-    </joint>
     <xacro:my_link
             name="tip_link"
@@ -187,9 +143,4 @@
             z="${tip_z}"
             m="${tip_m}"/>
-    <joint name="tip_to_padding" type="fixed">
-        <parent link="tip_link"/>
-        <child link="padding_link"/>
-        <origin xyz="-0.0125 -0.16 0"/>
-    </joint>
     <xacro:my_link
             name="padding_link"
@@ -204,14 +155,44 @@
             z="0.01"
             m="0.005"/>
-<!--    <actuator>
-        <motor name="holder_to_proximal"        gear="100" joint="holder_to_proximal" />
-        <motor name="proximal_to_intermediate"  gear="100" joint="proximal_to_intermediate" />
-        <motor name="intermediate_to_tip"       gear="100" joint="intermediate_to_tip" />
-    </actuator>-->
-<!--    <transmission name="holder_to_proximal">
-        <joint name="holder_to_proximal" />
-        <actuator name="holder_to_proximal">
-            <mechanicalReduction>50</mechanicalReduction>
-        </actuator>
-    </transmission> -->
+    <joint name="holder_joint" type="fixed">
+        <parent link="world"/>
+        <child link="holder_link"/>
+        <origin xyz="0 0 0" rpy="0 0 0"/>
+    </joint>
+    <joint name="holder_to_stage" type="fixed">
+        <parent link="holder_link"/>
+        <child link="stage_link"/>
+        <origin xyz="0 0 -0.2665"/>
+    </joint>
+    <joint name="holder_to_proximal" type="revolute">
+        <parent link="holder_link"/>
+        <child link="proximal_link"/>
+        <limit effort="1000" lower="0" upper="3.14159265359" velocity="1000"/>
+        <axis rpy="0 0 0" xyz="0 1 0"/>
+        <origin rpy="0 -1.5708 0" xyz="0 0 0"/>
+    </joint>
+    <joint name="holder_to_base" type="fixed">
+        <parent link="holder_link"/>
+        <child link="base_link"/>
+        <origin xyz="0 0.20595 0"/>
+    </joint>
+    <joint name="proximal_to_intermediate" type="revolute">
+        <parent link="proximal_link"/>
+        <child link="intermediate_link"/>
+        <limit effort="1000" lower="-5.846853" upper="0" velocity="1000"/>
+        <axis rpy="0 0 0" xyz="-1 0 0"/>
+        <origin rpy="2.9234265 0 0" xyz="0.014 0.02695 0"/>
+    </joint>
+    <joint name="intermediate_to_tip" type="revolute">
+        <parent link="intermediate_link"/>
+        <child link="tip_link"/>
+        <limit effort="1000" lower="0" upper="6.00394" velocity="1000"/>
+        <axis rpy="0 0 0" xyz="1 0 0"/>
+        <origin rpy="-2.9 0 0" xyz="0 -0.16 0"/>
+    </joint>
+    <joint name="tip_to_padding" type="fixed">
+        <parent link="tip_link"/>
+        <child link="padding_link"/>
+        <origin xyz="-0.0125 -0.16 0"/>
+    </joint>
 </robot>

Commit message: some further simplifications

File: xacro/manipulator.urdf.xacro (robot description, xacro)
@@ -5,7 +5,7 @@
        xmlns:sensor="http://playerstage.sourceforge.net/gazebo/xmlschema/#sensor"
        xmlns:xacro="http://playerstage.sourceforge.net/gazebo/xmlschema/#interface">
-    <xacro:property name="color_name" value="grey"/>
-    <xacro:property name="color" value="0.8 0.8 0.8"/>
-    <xacro:property name="opacity" value="0.8"/>
+    <xacro:property name="material_name" value="material"/>
+    <xacro:property name="color" value="0.6 0.6 1.0"/>
+    <xacro:property name="opacity" value="1.0"/>
     <!-- Meshes -->
     <xacro:property name="mesh_ext" value="stl"/>
@@ -37,6 +37,5 @@
     </mujoco>
     <xacro:macro name="my_link" params="name origin_rpy origin_xyz
-                                        mesh_file color_name color
-                                        opacity x y z m">
+                                        mesh_file x y z m">
         <link name="${name}">
             <inertial>
@@ -54,5 +53,5 @@
                     <mesh filename="${mesh_file}"/>
                 </geometry>
-                <material name="${color_name}">
+                <material name="${material_name}">
                     <color rgba="${color} ${opacity}"/>
                 </material>
@@ -63,5 +62,5 @@
                     <mesh filename="${mesh_file}"/>
                 </geometry>
-                <material name="${color_name}">
+                <material name="${material_name}">
                     <color rgba="${color} ${opacity}"/>
                 </material>
@@ -76,7 +75,4 @@
             origin_xyz="0 0 0"
             mesh_file="${holder_link_mesh}"
-            color_name="${color_name}"
-            color="${color}"
-            opacity="${opacity}"
             x="0.1"
             y="0.1"
@@ -88,7 +84,4 @@
             origin_xyz="0 0 0"
             mesh_file="${stage_link_mesh}"
-            color_name="${color_name}"
-            color="${color}"
-            opacity="${opacity}"
             x="0.5"
             y="0.5"
@@ -100,7 +93,4 @@
             origin_xyz="0 0 0"
             mesh_file="${proximal_link_mesh}"
-            color_name="${color_name}"
-            color="${color}"
-            opacity="${opacity}"
             x="${proximal_x}"
             y="${proximal_y}"
@@ -112,7 +102,4 @@
             origin_xyz="0 0 0"
             mesh_file="${intermediate_link_mesh}"
-            color_name="${color_name}"
-            color="${color}"
-            opacity="${opacity}"
             x="${intermediate_x}"
             y="${intermediate_y}"
@@ -124,7 +111,4 @@
             origin_xyz="0 0 0"
             mesh_file="${base_link_mesh}"
-            color_name="${color_name}"
-            color="${color}"
-            opacity="${opacity}"
             x="0.1"
             y="0.1"
@@ -136,7 +120,4 @@
             origin_xyz="0 0 0"
             mesh_file="${tip_link_mesh}"
-            color_name="${color_name}"
-            color="${color}"
-            opacity="${opacity}"
             x="${tip_x}"
             y="${tip_y}"
@@ -148,7 +129,4 @@
             origin_xyz="0 0 0"
             mesh_file="${padding_link_mesh}"
-            color_name="${color_name}"
-            color="${color}"
-            opacity="${opacity}"
             x="0.01"
             y="0.01"

Commit message: renaming

File: xacro/manipulator.urdf.xacro (robot description, xacro)
@@ -9,13 +9,13 @@
     <xacro:property name="opacity" value="1.0"/>
     <!-- Meshes -->
-    <xacro:property name="mesh_ext" value="stl"/>
-    <xacro:property name="mesh_dir" value="package://robot_properties_manipulator/meshes/${mesh_ext}"/>
-    <xacro:property name="stage_link_mesh" value="${mesh_dir}/Stage_simplified.${mesh_ext}"/>
-    <xacro:property name="base_link_mesh" value="${mesh_dir}/SIM__BL-Finger_Base.${mesh_ext}"/>
-    <xacro:property name="holder_link_mesh" value="${mesh_dir}/BL_Finger_Holder_SIM.${mesh_ext}"/>
-    <xacro:property name="proximal_link_mesh" value="${mesh_dir}/SIM__BL-Finger_Proximal.${mesh_ext}"/>
-    <xacro:property name="intermediate_link_mesh" value="${mesh_dir}/SIM__BL-Finger_Intermediate.${mesh_ext}"/>
-    <xacro:property name="tip_link_mesh" value="${mesh_dir}/SIM_BL_FINGER_TIP_LINK.${mesh_ext}"/>
-    <xacro:property name="padding_link_mesh" value="${mesh_dir}/finger_padding.${mesh_ext}"/>
+    <xacro:property name="mesh_file_extension" value="stl"/>
+    <xacro:property name="mesh_dir" value="package://robot_properties_manipulator/meshes/${mesh_file_extension}"/>
+    <xacro:property name="base_mesh" value="${mesh_dir}/SIM__BL-Finger_Base.${mesh_file_extension}"/>
+    <xacro:property name="base_holder_mesh" value="${mesh_dir}/BL_Finger_Holder_SIM.${mesh_file_extension}"/>
+    <xacro:property name="base_stage_mesh" value="${mesh_dir}/Stage_simplified.${mesh_file_extension}"/>
+    <xacro:property name="proximal_mesh" value="${mesh_dir}/SIM__BL-Finger_Proximal.${mesh_file_extension}"/>
+    <xacro:property name="central_mesh" value="${mesh_dir}/SIM__BL-Finger_Intermediate.${mesh_file_extension}"/>
+    <xacro:property name="distal_mesh" value="${mesh_dir}/SIM_BL_FINGER_TIP_LINK.${mesh_file_extension}"/>
+    <xacro:property name="distal_padding_mesh" value="${mesh_dir}/finger_padding.${mesh_file_extension}"/>
     <!-- Proximal link Inertia -->
     <xacro:property name="proximal_x" value="0.0399"/>
@@ -34,5 +34,5 @@
     <xacro:property name="tip_m" value="0.02" />
     <mujoco>
-        <compiler meshdir="../meshes/${mesh_ext}/" balanceinertia="true" discardvisual="false" />
+        <compiler meshdir="../meshes/${mesh_file_extension}/" balanceinertia="true" discardvisual="false" />
     </mujoco>
     <xacro:macro name="my_link" params="name origin_rpy origin_xyz
@@ -74,5 +74,5 @@
             origin_rpy="0 0 0"
             origin_xyz="0 0 0"
-            mesh_file="${holder_link_mesh}"
+            mesh_file="${base_holder_mesh}"
             x="0.1"
             y="0.1"
@@ -83,5 +83,5 @@
             origin_rpy="0 0 0"
             origin_xyz="0 0 0"
-            mesh_file="${stage_link_mesh}"
+            mesh_file="${base_stage_mesh}"
             x="0.5"
             y="0.5"
@@ -92,5 +92,5 @@
             origin_rpy="0 0 0"
             origin_xyz="0 0 0"
-            mesh_file="${proximal_link_mesh}"
+            mesh_file="${proximal_mesh}"
             x="${proximal_x}"
             y="${proximal_y}"
@@ -101,5 +101,5 @@
             origin_rpy="0 0 0"
             origin_xyz="0 0 0"
-            mesh_file="${intermediate_link_mesh}"
+            mesh_file="${central_mesh}"
             x="${intermediate_x}"
             y="${intermediate_y}"
@@ -110,5 +110,5 @@
             origin_rpy="0 0 0"
             origin_xyz="0 0 0"
-            mesh_file="${base_link_mesh}"
+            mesh_file="${base_mesh}"
             x="0.1"
             y="0.1"
@@ -119,5 +119,5 @@
             origin_rpy="0 0 0"
             origin_xyz="0 0 0"
-            mesh_file="${tip_link_mesh}"
+            mesh_file="${distal_mesh}"
             x="${tip_x}"
             y="${tip_y}"
@@ -128,5 +128,5 @@
             origin_rpy="0 0 0"
             origin_xyz="0 0 0"
-            mesh_file="${padding_link_mesh}"
+            mesh_file="${distal_padding_mesh}"
             x="0.01"
             y="0.01"

Commit message: some more cleanup

File: xacro/manipulator.urdf.xacro (robot description, xacro)
@@ -33,7 +33,26 @@
     <xacro:property name="tip_z" value="0.024" />
     <xacro:property name="tip_m" value="0.02" />
-    <mujoco>
-        <compiler meshdir="../meshes/${mesh_file_extension}/" balanceinertia="true" discardvisual="false" />
-    </mujoco>
+    <xacro:macro name="static_link" params="name origin_rpy origin_xyz mesh_file">
+        <link name="${name}">
+            <visual>
+                <origin rpy="${origin_rpy}" xyz="${origin_xyz}"/>
+                <geometry>
+                    <mesh filename="${mesh_file}"/>
+                </geometry>
+                <material name="${material_name}">
+                    <color rgba="${color} ${opacity}"/>
+                </material>
+            </visual>
+            <collision>
+                <origin rpy="${origin_rpy}" xyz="${origin_xyz}"/>
+                <geometry>
+                    <mesh filename="${mesh_file}"/>
+                </geometry>
+                <material name="${material_name}">
+                    <color rgba="${color} ${opacity}"/>
+                </material>
+            </collision>
+        </link>
+    </xacro:macro>
     <xacro:macro name="my_link" params="name origin_rpy origin_xyz
                                         mesh_file x y z m">
@@ -69,23 +88,19 @@
     </xacro:macro>
     <!-- World Link -->
-    <link name="world"/>
-    <xacro:my_link
+    <xacro:static_link
+            name="base_link"
+            origin_rpy="0 0 0"
+            origin_xyz="0 0 0"
+            mesh_file="${base_mesh}"/>
+    <xacro:static_link
             name="holder_link"
             origin_rpy="0 0 0"
             origin_xyz="0 0 0"
-            mesh_file="${base_holder_mesh}"
-            x="0.1"
-            y="0.1"
-            z="0.1"
-            m="0.1"/>
-    <xacro:my_link
+            mesh_file="${base_holder_mesh}"/>
+    <xacro:static_link
             name="stage_link"
             origin_rpy="0 0 0"
             origin_xyz="0 0 0"
-            mesh_file="${base_stage_mesh}"
-            x="0.5"
-            y="0.5"
-            z="0.1"
-            m="5"/>
+            mesh_file="${base_stage_mesh}"/>
     <xacro:my_link
             name="proximal_link"
@@ -107,13 +122,4 @@
             m="${intermediate_m}"/>
     <xacro:my_link
-            name="base_link"
-            origin_rpy="0 0 0"
-            origin_xyz="0 0 0"
-            mesh_file="${base_mesh}"
-            x="0.1"
-            y="0.1"
-            z="0.1"
-            m="0.1"/>
-    <xacro:my_link
             name="tip_link"
             origin_rpy="0 0 0"
@@ -133,9 +139,4 @@
             z="0.01"
             m="0.005"/>
-    <joint name="holder_joint" type="fixed">
-        <parent link="world"/>
-        <child link="holder_link"/>
-        <origin xyz="0 0 0" rpy="0 0 0"/>
-    </joint>
     <joint name="holder_to_stage" type="fixed">
         <parent link="holder_link"/>

Commit message: further cleaned urdf

File: xacro/manipulator.urdf.xacro (robot description, xacro)
@@ -33,4 +33,5 @@
     <xacro:property name="tip_z" value="0.024" />
     <xacro:property name="tip_m" value="0.02" />
+    <!-- Some macros for convenience -->
     <xacro:macro name="static_link" params="name origin_rpy origin_xyz mesh_file">
         <link name="${name}">
@@ -55,5 +56,5 @@
         </link>
     </xacro:macro>
-    <xacro:macro name="my_link" params="name origin_rpy origin_xyz
+    <xacro:macro name="dynamic_link" params="name origin_rpy origin_xyz
                                         mesh_file x y z m">
         <link name="${name}">
@@ -87,5 +88,5 @@
         </link>
     </xacro:macro>
-    <!-- World Link -->
+    <!-- base link -->
     <xacro:static_link
             name="base_link"
@@ -94,14 +95,25 @@
             mesh_file="${base_mesh}"/>
     <xacro:static_link
-            name="holder_link"
+            name="base_holder_link"
             origin_rpy="0 0 0"
             origin_xyz="0 0 0"
             mesh_file="${base_holder_mesh}"/>
     <xacro:static_link
-            name="stage_link"
+            name="base_stage_link"
             origin_rpy="0 0 0"
             origin_xyz="0 0 0"
             mesh_file="${base_stage_mesh}"/>
-    <xacro:my_link
+    <joint name="base_holder_to_stage" type="fixed">
+        <parent link="base_holder_link"/>
+        <child link="base_stage_link"/>
+        <origin xyz="0 0 -0.2665"/>
+    </joint>
+    <joint name="base_holder_to_base" type="fixed">
+        <parent link="base_holder_link"/>
+        <child link="base_link"/>
+        <origin xyz="0 0.20595 0"/>
+    </joint>
+    <!-- proximal link -->
+    <xacro:dynamic_link
             name="proximal_link"
             origin_rpy="0 0 0"
@@ -112,5 +124,6 @@
             z="${proximal_z}"
             m="${proximal_m}"/>
-    <xacro:my_link
+    <!-- central link -->
+    <xacro:dynamic_link
             name="intermediate_link"
             origin_rpy="0 0 0"
@@ -121,5 +134,6 @@
             z="${intermediate_z}"
             m="${intermediate_m}"/>
-    <xacro:my_link
+    <!-- distal link -->
+    <xacro:dynamic_link
             name="tip_link"
             origin_rpy="0 0 0"
@@ -130,5 +144,5 @@
             z="${tip_z}"
             m="${tip_m}"/>
-    <xacro:my_link
+    <xacro:dynamic_link
             name="padding_link"
             origin_rpy="0 0 0"
@@ -139,20 +153,16 @@
             z="0.01"
             m="0.005"/>
-    <joint name="holder_to_stage" type="fixed">
-        <parent link="holder_link"/>
-        <child link="stage_link"/>
-        <origin xyz="0 0 -0.2665"/>
+    <joint name="tip_to_padding" type="fixed">
+        <parent link="tip_link"/>
+        <child link="padding_link"/>
+        <origin xyz="-0.0125 -0.16 0"/>
     </joint>
+    <!-- kinematics -->
     <joint name="holder_to_proximal" type="revolute">
-        <parent link="holder_link"/>
+        <parent link="base_holder_link"/>
         <child link="proximal_link"/>
         <limit effort="1000" lower="0" upper="3.14159265359" velocity="1000"/>
         <axis rpy="0 0 0" xyz="0 1 0"/>
         <origin rpy="0 -1.5708 0" xyz="0 0 0"/>
-    </joint>
-    <joint name="holder_to_base" type="fixed">
-        <parent link="holder_link"/>
-        <child link="base_link"/>
-        <origin xyz="0 0.20595 0"/>
     </joint>
     <joint name="proximal_to_intermediate" type="revolute">
@@ -170,8 +180,3 @@
         <origin rpy="-2.9 0 0" xyz="0 -0.16 0"/>
     </joint>
-    <joint name="tip_to_padding" type="fixed">
-        <parent link="tip_link"/>
-        <child link="padding_link"/>
-        <origin xyz="-0.0125 -0.16 0"/>
-    </joint>
 </robot>
