Commit message: got rid of some redundant stuff

File: xacro/manipulator.urdf.xacro (robot description, xacro)
@@ -18,19 +18,4 @@
     <xacro:property name="distal_mesh" value="${mesh_dir}/SIM_BL_FINGER_TIP_LINK.${mesh_file_extension}"/>
     <xacro:property name="distal_padding_mesh" value="${mesh_dir}/finger_padding.${mesh_file_extension}"/>
-    <!-- Proximal link Inertia -->
-    <xacro:property name="proximal_x" value="0.0399"/>
-    <xacro:property name="proximal_y" value="0.2115"/>
-    <xacro:property name="proximal_z" value="0.047138" />
-    <xacro:property name="proximal_m" value="0.180" />
-    <!-- Intermediate link Inertia -->
-    <xacro:property name="intermediate_x" value="0.0419"/>
-    <xacro:property name="intermediate_y" value="0.206"/>
-    <xacro:property name="intermediate_z" value="0.044276" />
-    <xacro:property name="intermediate_m" value="0.180" />
-    <!-- Tip link Inertia -->
-    <xacro:property name="tip_x" value="0.027317"/>
-    <xacro:property name="tip_y" value="0.183"/>
-    <xacro:property name="tip_z" value="0.024" />
-    <xacro:property name="tip_m" value="0.02" />
     <!-- Some macros for convenience -->
     <xacro:macro name="static_link" params="name origin_rpy origin_xyz mesh_file">
@@ -120,8 +105,8 @@
             origin_xyz="0 0 0"
             mesh_file="${proximal_mesh}"
-            x="${proximal_x}"
-            y="${proximal_y}"
-            z="${proximal_z}"
-            m="${proximal_m}"/>
+            x="0.0399"
+            y="0.2115"
+            z="0.047138"
+            m="0.180"/>
     <!-- central link -->
     <xacro:dynamic_link
@@ -130,8 +115,8 @@
             origin_xyz="0 0 0"
             mesh_file="${central_mesh}"
-            x="${intermediate_x}"
-            y="${intermediate_y}"
-            z="${intermediate_z}"
-            m="${intermediate_m}"/>
+            x="0.0419"
+            y="0.206"
+            z="0.044276"
+            m="0.180"/>
     <!-- distal link -->
     <xacro:dynamic_link
@@ -140,17 +125,13 @@
             origin_xyz="0 0 0"
             mesh_file="${distal_mesh}"
-            x="${tip_x}"
-            y="${tip_y}"
-            z="${tip_z}"
-            m="${tip_m}"/>
-    <xacro:dynamic_link
+            x="0.027317"
+            y="0.183"
+            z="0.024"
+            m="0.02"/>
+    <xacro:static_link
             name="padding_link"
             origin_rpy="0 0 0"
             origin_xyz="0 0 0"
-            mesh_file="${distal_padding_mesh}"
-            x="0.01"
-            y="0.01"
-            z="0.01"
-            m="0.005"/>
+            mesh_file="${distal_padding_mesh}"/>
     <joint name="tip_to_padding" type="fixed">
         <parent link="tip_link"/>

Commit message: some further simplification with appropriate macros

File: xacro/manipulator.urdf.xacro (robot description, xacro)
@@ -19,25 +19,33 @@
     <xacro:property name="distal_padding_mesh" value="${mesh_dir}/finger_padding.${mesh_file_extension}"/>
     <!-- Some macros for convenience -->
-    <xacro:macro name="static_link" params="name origin_rpy origin_xyz mesh_file">
-        <link name="${name}">
-            <visual>
-                <origin rpy="${origin_rpy}" xyz="${origin_xyz}"/>
-                <geometry>
-                    <mesh filename="${mesh_file}"/>
-                </geometry>
-                <material name="${material_name}">
-                    <color rgba="${color} ${opacity}"/>
-                </material>
-            </visual>
-            <collision>
-                <origin rpy="${origin_rpy}" xyz="${origin_xyz}"/>
-                <geometry>
-                    <mesh filename="${mesh_file}"/>
-                </geometry>
-                <material name="${material_name}">
-                    <color rgba="${color} ${opacity}"/>
-                </material>
-            </collision>
-        </link>
+    <xacro:macro name="add_geometry" params="origin_rpy origin_xyz mesh_file">
+        <visual>
+            <origin rpy="${origin_rpy}" xyz="${origin_xyz}"/>
+            <geometry>
+                <mesh filename="${mesh_file}"/>
+            </geometry>
+            <material name="${material_name}">
+                <color rgba="${color} ${opacity}"/>
+            </material>
+        </visual>
+        <collision>
+            <origin rpy="${origin_rpy}" xyz="${origin_xyz}"/>
+            <geometry>
+                <mesh filename="${mesh_file}"/>
+            </geometry>
+            <material name="${material_name}">
+                <color rgba="${color} ${opacity}"/>
+            </material>
+        </collision>
+    </xacro:macro>
+    <xacro:macro name="add_inertia" params="x y z m">
+        <inertial>
+            <origin rpy="0 0 0" xyz="0 0 0"/>
+            <mass value="${m}"/>
+            <inertia ixx="${1./12. * m * (y*y + z*z)}"
+                        iyy="${1./12. * m * (x*x + z*z)}"
+                        izz="${1./12. * m * (x*x + y*y)}"
+                        ixy="0" ixz="0" iyz="0"/>
+        </inertial>
     </xacro:macro>
     <xacro:macro name="dynamic_link" params="name origin_rpy origin_xyz
@@ -50,6 +58,5 @@
                          iyy="${1./12. * m * (x*x + z*z)}"
                          izz="${1./12. * m * (x*x + y*y)}"
-                         ixy="0" ixz="0" iyz="0"
-                />
+                         ixy="0" ixz="0" iyz="0"/>
             </inertial>
             <visual>
@@ -74,19 +81,22 @@
     </xacro:macro>
     <!-- base link -->
-    <xacro:static_link
-            name="base_link"
+    <link name="base_link">
+        <xacro:add_geometry
             origin_rpy="0 0 0"
             origin_xyz="0 0 0"
             mesh_file="${base_mesh}"/>
-    <xacro:static_link
-            name="base_holder_link"
+    </link>
+    <link name="base_holder_link">
+        <xacro:add_geometry
             origin_rpy="0 0 0"
             origin_xyz="0 0 0"
             mesh_file="${base_holder_mesh}"/>
-    <xacro:static_link
-            name="base_stage_link"
+    </link>
+    <link name="base_stage_link">
+        <xacro:add_geometry
             origin_rpy="0 0 0"
             origin_xyz="0 0 0"
             mesh_file="${base_stage_mesh}"/>
+    </link>
     <joint name="base_holder_to_stage" type="fixed">
         <parent link="base_holder_link"/>
@@ -129,9 +139,10 @@
             z="0.024"
             m="0.02"/>
-    <xacro:static_link
-            name="padding_link"
+    <link name="padding_link">
+        <xacro:add_geometry
             origin_rpy="0 0 0"
             origin_xyz="0 0 0"
             mesh_file="${distal_padding_mesh}"/>
+    </link>
     <joint name="tip_to_padding" type="fixed">
         <parent link="tip_link"/>

Commit message: further simplification and clean up

File: xacro/manipulator.urdf.xacro (robot description, xacro)
@@ -49,35 +49,4 @@
         </inertial>
     </xacro:macro>
-    <xacro:macro name="dynamic_link" params="name origin_rpy origin_xyz
-                                        mesh_file x y z m">
-        <link name="${name}">
-            <inertial>
-                <origin rpy="0 0 0" xyz="0 0 0"/>
-                <mass value="${m}"/>
-                <inertia ixx="${1./12. * m * (y*y + z*z)}"
-                         iyy="${1./12. * m * (x*x + z*z)}"
-                         izz="${1./12. * m * (x*x + y*y)}"
-                         ixy="0" ixz="0" iyz="0"/>
-            </inertial>
-            <visual>
-                <origin rpy="${origin_rpy}" xyz="${origin_xyz}"/>
-                <geometry>
-                    <mesh filename="${mesh_file}"/>
-                </geometry>
-                <material name="${material_name}">
-                    <color rgba="${color} ${opacity}"/>
-                </material>
-            </visual>
-            <collision>
-                <origin rpy="${origin_rpy}" xyz="${origin_xyz}"/>
-                <geometry>
-                    <mesh filename="${mesh_file}"/>
-                </geometry>
-                <material name="${material_name}">
-                    <color rgba="${color} ${opacity}"/>
-                </material>
-            </collision>
-        </link>
-    </xacro:macro>
     <!-- base link -->
     <link name="base_link">
@@ -110,33 +79,39 @@
     </joint>
     <!-- proximal link -->
-    <xacro:dynamic_link
-            name="proximal_link"
+    <link name="proximal_link">
+        <xacro:add_geometry
             origin_rpy="0 0 0"
             origin_xyz="0 0 0"
-            mesh_file="${proximal_mesh}"
+            mesh_file="${proximal_mesh}"/>
+        <xacro:add_inertia
             x="0.0399"
             y="0.2115"
             z="0.047138"
             m="0.180"/>
+    </link>
     <!-- central link -->
-    <xacro:dynamic_link
-            name="intermediate_link"
+    <link name="intermediate_link">
+        <xacro:add_geometry
             origin_rpy="0 0 0"
             origin_xyz="0 0 0"
-            mesh_file="${central_mesh}"
+            mesh_file="${central_mesh}"/>
+        <xacro:add_inertia
             x="0.0419"
             y="0.206"
             z="0.044276"
             m="0.180"/>
+    </link>
     <!-- distal link -->
-    <xacro:dynamic_link
-            name="tip_link"
+    <link name="tip_link">
+        <xacro:add_geometry
             origin_rpy="0 0 0"
             origin_xyz="0 0 0"
-            mesh_file="${distal_mesh}"
+            mesh_file="${distal_mesh}"/>
+        <xacro:add_inertia
             x="0.027317"
             y="0.183"
             z="0.024"
             m="0.02"/>
+    </link>
     <link name="padding_link">
         <xacro:add_geometry

Commit message: some renaming of joints and links

File: xacro/manipulator.urdf.xacro (robot description, xacro)
@@ -91,5 +91,5 @@
     </link>
     <!-- central link -->
-    <link name="intermediate_link">
+    <link name="central_link">
         <xacro:add_geometry
             origin_rpy="0 0 0"
@@ -103,5 +103,5 @@
     </link>
     <!-- distal link -->
-    <link name="tip_link">
+    <link name="distal_link">
         <xacro:add_geometry
             origin_rpy="0 0 0"
@@ -114,5 +114,5 @@
             m="0.02"/>
     </link>
-    <link name="padding_link">
+    <link name="distal_padding_link">
         <xacro:add_geometry
             origin_rpy="0 0 0"
@@ -121,26 +121,26 @@
     </link>
     <joint name="tip_to_padding" type="fixed">
-        <parent link="tip_link"/>
-        <child link="padding_link"/>
+        <parent link="distal_link"/>
+        <child link="distal_padding_link"/>
         <origin xyz="-0.0125 -0.16 0"/>
     </joint>
     <!-- kinematics -->
-    <joint name="holder_to_proximal" type="revolute">
+    <joint name="base_proximal_joint" type="revolute">
         <parent link="base_holder_link"/>
         <child link="proximal_link"/>
-        <limit effort="1000" lower="0" upper="3.14159265359" velocity="1000"/>
+        <limit effort="1000" lower="0" upper="3.14" velocity="1000"/>
         <axis rpy="0 0 0" xyz="0 1 0"/>
         <origin rpy="0 -1.5708 0" xyz="0 0 0"/>
     </joint>
-    <joint name="proximal_to_intermediate" type="revolute">
+    <joint name="proximal_central_joint" type="revolute">
         <parent link="proximal_link"/>
-        <child link="intermediate_link"/>
+        <child link="central_link"/>
         <limit effort="1000" lower="-5.846853" upper="0" velocity="1000"/>
         <axis rpy="0 0 0" xyz="-1 0 0"/>
         <origin rpy="2.9234265 0 0" xyz="0.014 0.02695 0"/>
     </joint>
-    <joint name="intermediate_to_tip" type="revolute">
-        <parent link="intermediate_link"/>
-        <child link="tip_link"/>
+    <joint name="central_distal_joint" type="revolute">
+        <parent link="central_link"/>
+        <child link="distal_link"/>
         <limit effort="1000" lower="0" upper="6.00394" velocity="1000"/>
         <axis rpy="0 0 0" xyz="1 0 0"/>

Commit message: xacro clean now, need to fix inertias

File: xacro/manipulator.urdf.xacro (robot description, xacro)
@@ -11,5 +11,5 @@
     <xacro:property name="mesh_file_extension" value="stl"/>
     <xacro:property name="mesh_dir" value="package://robot_properties_manipulator/meshes/${mesh_file_extension}"/>
-    <xacro:property name="base_mesh" value="${mesh_dir}/SIM__BL-Finger_Base.${mesh_file_extension}"/>
+    <xacro:property name="base_module_mesh" value="${mesh_dir}/SIM__BL-Finger_Base.${mesh_file_extension}"/>
     <xacro:property name="base_holder_mesh" value="${mesh_dir}/BL_Finger_Holder_SIM.${mesh_file_extension}"/>
     <xacro:property name="base_stage_mesh" value="${mesh_dir}/Stage_simplified.${mesh_file_extension}"/>
@@ -54,11 +54,11 @@
             origin_rpy="0 0 0"
             origin_xyz="0 0 0"
-            mesh_file="${base_mesh}"/>
+            mesh_file="${base_holder_mesh}"/>
     </link>
-    <link name="base_holder_link">
+    <link name="base_module_link">
         <xacro:add_geometry
             origin_rpy="0 0 0"
             origin_xyz="0 0 0"
-            mesh_file="${base_holder_mesh}"/>
+            mesh_file="${base_module_mesh}"/>
     </link>
     <link name="base_stage_link">
@@ -68,12 +68,12 @@
             mesh_file="${base_stage_mesh}"/>
     </link>
-    <joint name="base_holder_to_stage" type="fixed">
-        <parent link="base_holder_link"/>
+    <joint name="base_to_stage" type="fixed">
+        <parent link="base_link"/>
         <child link="base_stage_link"/>
         <origin xyz="0 0 -0.2665"/>
     </joint>
-    <joint name="base_holder_to_base" type="fixed">
-        <parent link="base_holder_link"/>
-        <child link="base_link"/>
+    <joint name="base_to_module" type="fixed">
+        <parent link="base_link"/>
+        <child link="base_module_link"/>
         <origin xyz="0 0.20595 0"/>
     </joint>
@@ -127,5 +127,5 @@
     <!-- kinematics -->
     <joint name="base_proximal_joint" type="revolute">
-        <parent link="base_holder_link"/>
+        <parent link="base_link"/>
         <child link="proximal_link"/>
         <limit effort="1000" lower="0" upper="3.14" velocity="1000"/>

Commit message: set inertias and coms to something reasonable

File: xacro/manipulator.urdf.xacro (robot description, xacro)
@@ -39,12 +39,13 @@
         </collision>
     </xacro:macro>
-    <xacro:macro name="add_inertia" params="x y z m">
+    <xacro:macro name="add_inertia" params="length_x length_y length_z mass com">
         <inertial>
-            <origin rpy="0 0 0" xyz="0 0 0"/>
-            <mass value="${m}"/>
-            <inertia ixx="${1./12. * m * (y*y + z*z)}"
-                        iyy="${1./12. * m * (x*x + z*z)}"
-                        izz="${1./12. * m * (x*x + y*y)}"
-                        ixy="0" ixz="0" iyz="0"/>
+            <origin rpy="0 0 0" xyz="${com}"/>
+            <mass value="${mass}"/>
+            <inertia
+                    ixx="${1./12. * mass * (length_y*length_y + length_z*length_z)}"
+                    iyy="${1./12. * mass * (length_x*length_x + length_z*length_z)}"
+                    izz="${1./12. * mass * (length_x*length_x + length_y*length_y)}"
+                    ixy="0" ixz="0" iyz="0"/>
         </inertial>
     </xacro:macro>
@@ -85,8 +86,9 @@
             mesh_file="${proximal_mesh}"/>
         <xacro:add_inertia
-            x="0.0399"
-            y="0.2115"
-            z="0.047138"
-            m="0.180"/>
+            length_x="0.04"
+            length_y="0.2"
+            length_z="0.04"
+            mass="0.2"
+            com="0 0.1 0"/>
     </link>
     <!-- central link -->
@@ -97,8 +99,9 @@
             mesh_file="${central_mesh}"/>
         <xacro:add_inertia
-            x="0.0419"
-            y="0.206"
-            z="0.044276"
-            m="0.180"/>
+            length_x="0.04"
+            length_y="0.2"
+            length_z="0.04"
+            mass="0.2"
+            com="0 -0.1 0"/>
     </link>
     <!-- distal link -->
@@ -109,8 +112,9 @@
             mesh_file="${distal_mesh}"/>
         <xacro:add_inertia
-            x="0.027317"
-            y="0.183"
-            z="0.024"
-            m="0.02"/>
+            length_x="0.02"
+            length_y="0.2"
+            length_z="0.02"
+            mass="0.05"
+            com="0 -0.1 0"/>
     </link>
     <link name="distal_padding_link">
