Commit message: Add tip padding to lower link and rename tip link
Add the mesh of the tip padding to the lower link instead of the padding
link.  This way, there is no collision between the meshes of the two
links.

Keep the tip link (which does not have any geometry anymore) as it is
useful to get the tip position.  However, rename it to
`finger_tip_link`, i.e. remove the "padding" from the name.

File: xacro/finger.urdf.xacro (robot description, xacro)
@@ -85,4 +85,8 @@
             origin_xyz="${mesh_x_offset} 0 0"
             mesh_file="${lower_link_mesh}"/>
+        <xacro:add_geometry
+            origin_rpy="0 0 0"
+            origin_xyz="0 0 -${lower_joint_to_tip_distance}"
+            mesh_file="${tip_padding_mesh}"/>
         <xacro:add_inertia
             length_x="0.01"
@@ -92,14 +96,9 @@
             com="0 0 -0.07"/>
     </link>
-    <!-- fixed link for padding around the finger tip -->
-    <link name="finger_tip_padding_link">
-        <xacro:add_geometry
-            origin_rpy="0 0 0"
-            origin_xyz="0 0 0"
-            mesh_file="${tip_padding_mesh}"/>
-    </link>
-    <joint name="finger_lower_to_padding_joint" type="fixed">
+    <!-- fixed link for finger tip -->
+    <link name="finger_tip_link" />
+    <joint name="finger_lower_to_tip_joint" type="fixed">
         <parent link="finger_lower_link"/>
-        <child link="finger_tip_padding_link"/>
+        <child link="finger_tip_link"/>
         <origin xyz="0 0 -${lower_joint_to_tip_distance}"/>
     </joint>

Commit message: added 3-finger urdf

File: xacro/finger.urdf.xacro (robot description, xacro)
@@ -8,124 +8,7 @@
     finger tip which should make it easy to place the finger in the world.
     -->
-    <xacro:include filename="macros.xacro" />
-    <!-- Meshes -->
-    <xacro:property name="mesh_file_extension" value="stl"/>
-    <xacro:property name="mesh_dir" value="package://robot_properties_manipulator/meshes/${mesh_file_extension}"/>
-    <xacro:property name="upper_base_mesh" value="${mesh_dir}/SIM__BL-Finger_Base.${mesh_file_extension}"/>
-    <xacro:property name="base_holder_mesh" value="${mesh_dir}/BL_Finger_Holder_SIM.${mesh_file_extension}"/>
-    <xacro:property name="upper_link_mesh" value="${mesh_dir}/SIM__BL-Finger_Proximal.${mesh_file_extension}"/>
-    <xacro:property name="middle_link_mesh" value="${mesh_dir}/SIM__BL-Finger_Intermediate.${mesh_file_extension}"/>
-    <xacro:property name="lower_link_mesh" value="${mesh_dir}/SIM_BL_FINGER_TIP_LINK.${mesh_file_extension}"/>
-    <xacro:property name="tip_padding_mesh" value="${mesh_dir}/finger_padding.${mesh_file_extension}"/>
-    <!-- Distance from outer edge of the link to the joint center -->
-    <xacro:property name="upper_joint_center_offset" value="0.02695" />
-    <xacro:property name="upper_link_length" value="0.179" />
-    <xacro:property name="middle_to_lower_joint_distance" value="0.16" />
-    <xacro:property name="lower_joint_to_tip_distance" value="0.16" />
-    <xacro:property name="mesh_x_offset" value="0.014" />
+    <xacro:include filename="finger_macro.urdf.xacro" />
     <!--
     Fixed links for the finger base (parts where the upper link is mounted).
     -->
-    <link name="finger_base_link">
-        <xacro:add_geometry
-            origin_rpy="0 0 0"
-            origin_xyz="0 ${upper_link_length} 0"
-            mesh_file="${upper_base_mesh}"/>
-    </link>
-    <link name="finger_upper_holder_link">
-        <xacro:add_geometry
-            origin_rpy="0 0 0"
-            origin_xyz="0 0 0"
-            mesh_file="${base_holder_mesh}"/>
-        <!--
-          for some reason this link needs to have some inertia defined,
-          otherwise the model won't show up in gazebo.
-        -->
-        <xacro:add_inertia
-            length_x="0.05"
-            length_y="0.05"
-            length_z="0.05"
-            mass="0.5"
-            com="0 0 0"/>
-    </link>
-    <joint name="finger_base_to_holder" type="fixed">
-        <parent link="finger_base_link"/>
-        <child link="finger_upper_holder_link"/>
-        <origin xyz="0 -${upper_joint_center_offset} 0" rpy="0 0 0" />
-    </joint>
-    <!-- The movable links (upper, middle and lower) of the finger. -->
-    <!-- TODO inertia parameters don't look correct, they cant be same for upper and middle! -->
-    <link name="finger_upper_link">
-        <xacro:add_geometry
-            origin_rpy="0 0 0"
-            origin_xyz="0 -${upper_joint_center_offset} 0"
-            mesh_file="${upper_link_mesh}"/>
-        <xacro:add_inertia
-            length_x="0.02"
-            length_y="0.14"
-            length_z="0.02"
-            mass="0.2"
-            com="0 0.06 0"/>
-    </link>
-    <link name="finger_middle_link">
-        <xacro:add_geometry
-            origin_rpy="${pi/2} 0 0"
-            origin_xyz="${mesh_x_offset} 0 0"
-            mesh_file="${middle_link_mesh}"/>
-        <xacro:add_inertia
-            length_x="0.02"
-            length_y="0.02"
-            length_z="0.14"
-            mass="0.2"
-            com="${2 * mesh_x_offset} 0 -0.06"/>
-    </link>
-    <link name="finger_lower_link">
-        <xacro:add_geometry
-            origin_rpy="${pi/2} 0 0"
-            origin_xyz="${mesh_x_offset} 0 0"
-            mesh_file="${lower_link_mesh}"/>
-        <xacro:add_geometry
-            origin_rpy="0 0 0"
-            origin_xyz="0 0 -${lower_joint_to_tip_distance}"
-            mesh_file="${tip_padding_mesh}"/>
-        <xacro:add_inertia
-            length_x="0.01"
-            length_y="0.01"
-            length_z="0.14"
-            mass="0.05"
-            com="0 0 -0.07"/>
-    </link>
-    <!-- fixed link for finger tip -->
-    <link name="finger_tip_link" />
-    <joint name="finger_lower_to_tip_joint" type="fixed">
-        <parent link="finger_lower_link"/>
-        <child link="finger_tip_link"/>
-        <origin xyz="0 0 -${lower_joint_to_tip_distance}"/>
-    </joint>
-    <!-- kinematics -->
-    <!-- TODO: joint limits are based on values from wiki
-    (https://atlas.is.localnet/confluence/display/AMDW/Forward+Kinematics) but
-    should be verified on the real system (especially the finger tip limits look
-    a bit too big when visualizing the model. -->
-    <joint name="finger_base_to_upper_joint" type="revolute">
-        <parent link="finger_base_link"/>
-        <child link="finger_upper_link"/>
-        <limit effort="1000" lower="-${pi/2}" upper="${pi/2}" velocity="1000"/>
-        <axis xyz="0 1 0"/>
-        <origin rpy="0 0 0" xyz="0 0 0"/>
-    </joint>
-    <joint name="finger_upper_to_middle_joint" type="revolute">
-        <parent link="finger_upper_link"/>
-        <child link="finger_middle_link"/>
-        <limit effort="1000" lower="${radians(-77.5)}" upper="${radians(257.5)}" velocity="1000"/>
-        <axis xyz="-1 0 0"/>
-        <origin rpy="0 0 0" xyz="0 0 0"/>
-    </joint>
-    <joint name="finger_middle_to_lower_joint" type="revolute">
-        <parent link="finger_middle_link"/>
-        <child link="finger_lower_link"/>
-        <limit effort="1000" lower="${radians(-172)}" upper="${radians(172)}" velocity="1000"/>
-        <axis xyz="1 0 0"/>
-        <origin rpy="0 0 0" xyz="0 0 -${middle_to_lower_joint_distance}"/>
-    </joint>
 </robot>

File: xacro/macros.xacro (robot description, xacro)
@@ -5,9 +5,9 @@
     <xacro:property name="color" value="0.6 0.6 1.0"/>
     <xacro:property name="opacity" value="1.0"/>
-    <xacro:macro name="add_geometry" params="origin_rpy origin_xyz mesh_file">
+    <xacro:macro name="add_geometry" params="origin_rpy origin_xyz mesh_file mesh_scale:='1 1 1'">
         <visual>
             <origin rpy="${origin_rpy}" xyz="${origin_xyz}"/>
             <geometry>
-                <mesh filename="${mesh_file}"/>
+                <mesh scale="${mesh_scale}" filename="${mesh_file}"/>
             </geometry>
             <material name="${material_name}">

Commit message: updated after changing 'idx', 'mesh_scale', and variable names

File: xacro/finger.urdf.xacro (robot description, xacro)
@@ -10,7 +10,7 @@
     <xacro:include filename="finger_macro.urdf.xacro" />
     <!--
-    Simply calling the "finger" macro (without passing any idx) implies a call for single finger.
+    Simply calling the "finger" macro (without passing any suffix) implies a call for single finger.
     The parameters are automatically set inside the finger_macro file, to accomodate for single finger.
     -->
-    <finger/>
+    <xacro:finger/>
 </robot>

File: xacro/finger_macro.urdf.xacro (robot description, xacro)
@@ -1,4 +1,4 @@
 <?xml version="1.0" ?>
-<robot name="finger" xmlns:xacro="https://ei.is.tuebingen.mpg.de/xacro">
+<robot xmlns:xacro="https://ei.is.tuebingen.mpg.de/xacro">
     <!--
     Frames are defined such that they all align with the base frame when all
@@ -25,24 +25,28 @@
     <xacro:property name="mesh_x_offset" value="0.014" />
     <xacro:property name="centre_offset" value="0.014" />
-    <xacro:property name="lower_link_mesh_scale" value="0.001 0.001 0.001" />
-    <xacro:property name="tip_padding" value="0" />
-    <xacro:property name="base_holder" value="0" />
+    <!--
+    ROS uses meters for length. Since the new lower_link_mesh and the stage_mesh is made using millimeters as units,
+    scaling them down to 1/1000 of their current size loads them with the correct size.
+    -->
+    <xacro:property name="lower_link_mesh_scale" value="0.001" />
+    <xacro:property name="tip_padding" value="0" /> <!-- if this flag is set to 1 (True), finger padding is added at the finger tips -->
+    <xacro:property name="base_holder" value="0" /> <!-- if this flag is set to 1 (True), an upper base_holder is added -->
     <!--
     Defining the "finger" macro which is used for both single and tri-finger.
-    The macro takes "idx" as a parameter for the three fingers.
-    In case of single finger, no "idx" value is passed.
+    The macro takes "suffix" as a parameter to differentiate between multiple fingers
+    In case of single finger, no "suffix" value is passed.
     -->
-    <xacro:macro name="finger" params="idx:=''">
-        <!-- In case of single finger (i.e. when no idx is passed), we change the default values of the following variables. -->
-        <xacro:if value="${idx == ''}">
-            <xacro:property name="lower_link_mesh" value="${mesh_dir}/SIM_BL_FINGER_TIP_LINK.${mesh_file_extension}"/> <!-- mesh for single finger -->
-            <xacro:property name="lower_link_mesh_scale" value="1 1 1" /> <!-- lower_link_mesh has different scale for single and 3-finger -->
-            <xacro:property name="tip_padding" value="1" /> <!-- Flag for tip_padding. 1 = True -->
-            <xacro:property name="base_holder" value="1" /> <!-- Flag for upper base_holder. 1 = True -->
+    <xacro:macro name="finger" params="suffix:=''">
+        <!-- In case of single finger (i.e. when no suffix is passed), we change the default values of the following variables. -->
+        <xacro:if value="${suffix == ''}">
+            <xacro:property name="lower_link_mesh" value="${mesh_dir}/SIM_BL_FINGER_TIP_LINK.${mesh_file_extension}"/> <!-- lower_link_mesh for single finger -->
+            <xacro:property name="lower_link_mesh_scale" value="1" /> <!-- not changing the scale here. Therefore, keeping the value to 1 (original scale) -->
+            <xacro:property name="tip_padding" value="1" />
+            <xacro:property name="base_holder" value="1" />
         </xacro:if>
         <!--
         Fixed links for the finger base (parts where the upper link is mounted).
         -->
-        <link name="finger_base_link${idx}">
+        <link name="finger_base_link${suffix}">
             <xacro:add_geometry
                 origin_rpy="0 0 0"
@@ -51,5 +55,5 @@
         </link>
         <xacro:if value="${base_holder == 1}"> <!-- base_holder is added in case of single finger -->
-            <link name="finger_upper_holder_link${idx}">
+            <link name="finger_upper_holder_link${suffix}">
                 <xacro:add_geometry
                     origin_rpy="0 0 0"
@@ -67,7 +71,7 @@
                     com="0 0 0"/>
             </link>
-            <joint name="finger_base_to_holder${idx}" type="fixed">
-                <parent link="finger_base_link${idx}"/>
-                <child link="finger_upper_holder_link${idx}"/>
+            <joint name="finger_base_to_holder${suffix}" type="fixed">
+                <parent link="finger_base_link${suffix}"/>
+                <child link="finger_upper_holder_link${suffix}"/>
                 <origin xyz="0 -${upper_joint_center_offset} 0" rpy="0 0 0" />
             </joint>
@@ -75,5 +79,5 @@
         <!-- The movable links (upper, middle and lower) of the finger. -->
         <!-- TODO inertia parameters don't look correct, they cant be same for upper and middle! -->
-        <link name="finger_upper_link${idx}">
+        <link name="finger_upper_link${suffix}">
             <xacro:add_geometry
                 origin_rpy="0 0 0"
@@ -87,5 +91,5 @@
                 com="0 0.06 0"/>
         </link>
-        <link name="finger_middle_link${idx}">
+        <link name="finger_middle_link${suffix}">
             <xacro:add_geometry
                 origin_rpy="${pi/2} 0 0"
@@ -99,5 +103,5 @@
                 com="${2 * mesh_x_offset} 0 -0.06"/>
         </link>
-        <link name="finger_lower_link${idx}">
+        <link name="finger_lower_link${suffix}">
             <xacro:add_geometry
                 origin_rpy="${pi/2} 0 0"
@@ -119,8 +123,8 @@
         </link>
         <!-- fixed link for finger tip -->
-        <link name="finger_tip_link${idx}" />
-        <joint name="finger_lower_to_tip_joint${idx}" type="fixed">
-            <parent link="finger_lower_link${idx}"/>
-            <child link="finger_tip_link${idx}"/>
+        <link name="finger_tip_link${suffix}" />
+        <joint name="finger_lower_to_tip_joint${suffix}" type="fixed">
+            <parent link="finger_lower_link${suffix}"/>
+            <child link="finger_tip_link${suffix}"/>
             <origin xyz="0 0 -${lower_joint_to_tip_distance}"/>
         </joint>
@@ -130,21 +134,21 @@
         should be verified on the real system (especially the finger tip limits look
         a bit too big when visualizing the model. -->
-        <joint name="finger_base_to_upper_joint${idx}" type="revolute">
-            <parent link="finger_base_link${idx}"/>
-            <child link="finger_upper_link${idx}"/>
+        <joint name="finger_base_to_upper_joint${suffix}" type="revolute">
+            <parent link="finger_base_link${suffix}"/>
+            <child link="finger_upper_link${suffix}"/>
             <limit effort="1000" lower="-${pi/2}" upper="${pi/2}" velocity="1000"/>
             <axis xyz="0 1 0"/>
             <origin rpy="0 0 0" xyz="0 0 0"/>
         </joint>
-        <joint name="finger_upper_to_middle_joint${idx}" type="revolute">
-            <parent link="finger_upper_link${idx}"/>
-            <child link="finger_middle_link${idx}"/>
+        <joint name="finger_upper_to_middle_joint${suffix}" type="revolute">
+            <parent link="finger_upper_link${suffix}"/>
+            <child link="finger_middle_link${suffix}"/>
             <limit effort="1000" lower="${radians(-77.5)}" upper="${radians(257.5)}" velocity="1000"/>
             <axis xyz="-1 0 0"/>
             <origin rpy="0 0 0" xyz="0 0 0"/>
         </joint>
-        <joint name="finger_middle_to_lower_joint${idx}" type="revolute">
-            <parent link="finger_middle_link${idx}"/>
-            <child link="finger_lower_link${idx}"/>
+        <joint name="finger_middle_to_lower_joint${suffix}" type="revolute">
+            <parent link="finger_middle_link${suffix}"/>
+            <child link="finger_lower_link${suffix}"/>
             <limit effort="1000" lower="${radians(-172)}" upper="${radians(172)}" velocity="1000"/>
             <axis xyz="1 0 0"/>

File: xacro/macros.xacro (robot description, xacro)
@@ -5,9 +5,9 @@
     <xacro:property name="color" value="0.6 0.6 1.0"/>
     <xacro:property name="opacity" value="1.0"/>
-    <xacro:macro name="add_geometry" params="origin_rpy origin_xyz mesh_file mesh_scale:='1 1 1'">
+    <xacro:macro name="add_geometry" params="origin_rpy origin_xyz mesh_file mesh_scale:='1'">
         <visual>
             <origin rpy="${origin_rpy}" xyz="${origin_xyz}"/>
             <geometry>
-                <mesh scale="${mesh_scale}" filename="${mesh_file}"/>
+                <mesh scale="${mesh_scale} ${mesh_scale} ${mesh_scale}" filename="${mesh_file}"/>
             </geometry>
             <material name="${material_name}">

File: xacro/trifinger_with_stage.urdf.xacro (robot description, xacro)
@@ -4,5 +4,7 @@
     <xacro:include filename="finger_macro.urdf.xacro" />
     <xacro:include filename="macros.xacro" />
-    <!-- Add the "stage" -->
+    <!-- Define the global base_link and place all other objects relative to it. -->
+    <link name="base_link" />
+    <!-- Adding the "stage" -->
     <!-- Meshes -->
     <xacro:property name="mesh_file_extension" value="stl"/>
@@ -14,9 +16,10 @@
             origin_xyz="0 0 0"
             mesh_file="${stage_mesh}"
-            mesh_scale="0.001 0.001 0.001"/>
+            mesh_scale="0.001"/>
+            <!--
+            ROS uses meters for length. Since the new lower_link_mesh and the stage_mesh is made using millimeters as units,
+            scaling them down to 1/1000 of their current size loads them with the correct size.
+            -->
     </link>
-    <!-- Finished adding the stage -->
-    <!-- Define the global base_link and place stage relative to it. -->
-    <link name="base_link" />
     <!-- Define the stage -->
     <joint name="base_to_stage" type="fixed">
@@ -33,25 +36,25 @@
     </joint>
     <!-- Define the three fingers and place them relative to the upper holder -->
-    <finger idx="_0"/>
-    <finger idx="_120"/>
-    <finger idx="_240"/>
-    <xacro:property name="offset" value="0.04"/>
-    <xacro:property name="angle1" value="${radians(0)}"/>
-    <xacro:property name="angle2" value="${radians(120)}"/>
-    <xacro:property name="angle3" value="${radians(240)}"/>
+    <xacro:finger suffix="_0"/>
+    <xacro:finger suffix="_120"/>
+    <xacro:finger suffix="_240"/>
+    <xacro:property name="offset" value="0.04"/> <!-- upper_holder to finger offset -->
+    <xacro:property name="angle_0" value="${radians(0)}"/>
+    <xacro:property name="angle_120" value="${radians(120)}"/>
+    <xacro:property name="angle_240" value="${radians(240)}"/>
     <joint name="holder_to_finger_0" type="fixed">
         <parent link="upper_holder_link"/>
         <child link="finger_base_link_0"/>
-        <origin xyz="${offset * sin(angle1)} ${offset * cos(angle1)} 0" rpy="0 0 0"/>
+        <origin xyz="${offset * sin(angle_0)} ${offset * cos(angle_0)} 0" rpy="0 0 0"/>
     </joint>
-    <joint name="holder_to_finger_1" type="fixed">
+    <joint name="holder_to_finger_120" type="fixed">
         <parent link="upper_holder_link"/>
         <child link="finger_base_link_120"/>
-        <origin xyz="${offset * sin(angle2)} ${offset * cos(angle2)} 0" rpy="0 0 ${radians(240)}"/>
+        <origin xyz="${offset * sin(angle_120)} ${offset * cos(angle_120)} 0" rpy="0 0 -${angle_120}"/>
     </joint>
-    <joint name="holder_to_finger_2" type="fixed">
+    <joint name="holder_to_finger_240" type="fixed">
         <parent link="upper_holder_link"/>
         <child link="finger_base_link_240"/>
-        <origin xyz="${offset * sin(angle3)} ${offset * cos(angle3)} 0" rpy="0 0 ${radians(120)}"/>
+        <origin xyz="${offset * sin(angle_240)} ${offset * cos(angle_240)} 0" rpy="0 0 -${angle_240}"/>
     </joint>
 </robot>

Commit message: Moving the definitions of the base link and base to finger_base joint to the finger xacro

File: xacro/finger.urdf.xacro (robot description, xacro)
@@ -14,3 +14,12 @@
     -->
     <xacro:finger/>
+    <!--
+    Define the global base link and place the finger relative to it.
+    -->
+    <link name="base_link" />
+    <joint name="base_to_finger" type="fixed">
+        <parent link="base_link"/>
+        <child link="finger_base_link"/>
+        <origin xyz="0 0 0.34"/>
+    </joint>
 </robot>

File: xacro/finger_macro.urdf.xacro (robot description, xacro)
@@ -32,4 +32,5 @@
     <xacro:property name="tip_padding" value="0" /> <!-- if this flag is set to 1 (True), finger padding is added at the finger tips -->
     <xacro:property name="base_holder" value="0" /> <!-- if this flag is set to 1 (True), an upper base_holder is added -->
+    <xacro:property name="tip_mass" value="0.075" />
     <!--
     Defining the "finger" macro which is used for both single and tri-finger.
@@ -44,4 +45,5 @@
             <xacro:property name="tip_padding" value="1" />
             <xacro:property name="base_holder" value="1" />
+            <xacro:property name="tip_mass" value="0.025" />
         </xacro:if>
         <!--
@@ -123,5 +125,12 @@
         </link>
         <!-- fixed link for finger tip -->
-        <link name="finger_tip_link${suffix}" />
+        <link name="finger_tip_link${suffix}">
+            <xacro:add_inertia
+                length_x="0.01"
+                length_y="0.01"
+                length_z="0.01"
+                com="0 0 0"
+                mass="${tip_mass}"/>
+        </link>
         <joint name="finger_lower_to_tip_joint${suffix}" type="fixed">
             <parent link="finger_lower_link${suffix}"/>

File: xacro/finger_with_stage.urdf.xacro (robot description, xacro)
@@ -4,11 +4,5 @@
     <xacro:include filename="finger.urdf.xacro" />
     <xacro:include filename="stage.urdf.xacro" />
-    <!-- Define the global base_link and place finger and stage relative to it. -->
-    <link name="base_link" />
-    <joint name="base_to_finger" type="fixed">
-        <parent link="base_link"/>
-        <child link="finger_base_link"/>
-        <origin xyz="0 0 0.34"/>
-    </joint>
+    <!-- Place the stage relative to the global base link. -->
     <joint name="base_to_stage" type="fixed">
         <parent link="base_link"/>
