Commit message: Inertias for base/finger_base/stage

File: xacro/finger.urdf.xacro (robot description, xacro)
@@ -17,5 +17,12 @@
     Define the global base link and place the finger relative to it.
     -->
-    <link name="base_link" />
+    <link name="base_link">
+      <xacro:add_inertia
+          length_x="0.005"
+          length_y="0.005"
+          length_z="0.005"
+          mass="1"
+          com="0 0 0"/>
+    </link>
     <joint name="base_to_finger" type="fixed">
         <parent link="base_link"/>

File: xacro/finger_macro.urdf.xacro (robot description, xacro)
@@ -55,4 +55,10 @@
                 origin_xyz="0 ${upper_link_length} 0"
                 mesh_file="${upper_base_mesh}"/>
+            <xacro:add_inertia
+                length_x="0.05"
+                length_y="0.05"
+                length_z="0.05"
+                mass="1"
+                com="0 0 0"/>
         </link>
         <xacro:if value="${base_holder == 1}"> <!-- base_holder is added in case of single finger -->

File: xacro/stage.urdf.xacro (robot description, xacro)
@@ -12,4 +12,10 @@
             origin_xyz="0 0 0"
             mesh_file="${stage_mesh}"/>
+        <xacro:add_inertia
+            length_x="0.3"
+            length_y="0.3"
+            length_z="0.05"
+            mass="1"
+            com="0 0 0"/>
     </link>
 </robot>

File: xacro/trifinger.urdf.xacro (robot description, xacro)
@@ -5,5 +5,12 @@
     <xacro:include filename="macros.xacro" />
     <!-- Define the global base_link and place all other objects relative to it. -->
-    <link name="base_link" />
+    <link name="base_link">
+      <xacro:add_inertia
+          length_x="0.005"
+          length_y="0.005"
+          length_z="0.005"
+          mass="1"
+          com="0 0 0"/>
+    </link>
     <!-- Define the upper holder -->
     <link name="upper_holder_link" />

File: xacro/trifinger_with_stage.urdf.xacro (robot description, xacro)
@@ -15,4 +15,10 @@
             mesh_file="${stage_mesh}"
             mesh_scale="1"/>
+        <xacro:add_inertia
+            length_x="0.3"
+            length_y="0.3"
+            length_z="0.05"
+            mass="1"
+            com="0 0 0"/>
             <!--
             ROS uses meters for length. Since the new lower_link_mesh and the stage_mesh is made using millimeters as units,

Commit message: Set different colours for the fingers
Add a "material" option to creating visuals and fingers.  This way the
three fingers of the TriFinger can be assigned different colours (0:
red, 120: green, 240: blue) to easily distinguish them.

Unfortunately I did not find a way to have a default material (defining
it in the macros file will lead to name collisions when including it
multiple times...), so this is a mandatory argument now.

File: xacro/finger.urdf.xacro (robot description, xacro)
@@ -9,9 +9,12 @@
     -->
     <xacro:include filename="finger_macro.urdf.xacro" />
+    <material name="finger_material">
+        <color rgba="0.6 0.6 0.6 1.0" />
+    </material>
     <!--
     Simply calling the "finger" macro (without passing any suffix) implies a call for single finger.
     The parameters are automatically set inside the finger_macro file, to accomodate for single finger.
     -->
-    <xacro:finger/>
+    <xacro:finger material="finger_material" />
     <!--
     Define the global base link and place the finger relative to it.

File: xacro/finger_macro.urdf.xacro (robot description, xacro)
@@ -38,5 +38,5 @@
     In case of single finger, no "suffix" value is passed.
     -->
-    <xacro:macro name="finger" params="suffix:=''">
+    <xacro:macro name="finger" params="material suffix:=''">
         <!-- In case of single finger (i.e. when no suffix is passed), we change the default values of the following variables. -->
         <xacro:if value="${suffix == ''}">
@@ -54,5 +54,6 @@
                 origin_rpy="0 0 0"
                 origin_xyz="0 ${upper_link_length} 0"
-                mesh_file="${upper_base_mesh}"/>
+                mesh_file="${upper_base_mesh}"
+                material="${material}" />
             <xacro:add_inertia
                 length_x="0.05"
@@ -67,5 +68,6 @@
                     origin_rpy="0 0 0"
                     origin_xyz="0 0 0"
-                    mesh_file="${base_holder_mesh}"/>
+                    mesh_file="${base_holder_mesh}"
+                    material="${material}" />
                 <!--
                   for some reason this link needs to have some inertia defined,
@@ -91,5 +93,6 @@
                 origin_rpy="0 0 0"
                 origin_xyz="0 -${upper_joint_center_offset} 0"
-                mesh_file="${upper_link_mesh}"/>
+                mesh_file="${upper_link_mesh}"
+                material="${material}" />
             <xacro:add_inertia
                 length_x="0.02"
@@ -103,5 +106,6 @@
                 origin_rpy="${pi/2} 0 0"
                 origin_xyz="${mesh_x_offset} 0 0"
-                mesh_file="${middle_link_mesh}"/>
+                mesh_file="${middle_link_mesh}"
+                material="${material}" />
             <xacro:add_inertia
                 length_x="0.02"
@@ -116,10 +120,12 @@
                 origin_xyz="${mesh_x_offset} 0 0"
                 mesh_file="${lower_link_mesh}"
-                mesh_scale="${lower_link_mesh_scale}"/>
+                mesh_scale="${lower_link_mesh_scale}"
+                material="${material}" />
             <xacro:if value="${tip_padding == 1}"> <!-- tip_padding is added in case of single finger -->
                 <xacro:add_geometry
                     origin_rpy="0 0 0"
                     origin_xyz="0 0 -${lower_joint_to_tip_distance}"
-                    mesh_file="${tip_padding_mesh}"/>
+                    mesh_file="${tip_padding_mesh}"
+                    material="${material}" />
             </xacro:if>
             <xacro:add_inertia

File: xacro/macros.xacro (robot description, xacro)
@@ -2,8 +2,6 @@
 <!-- Some macros for convenience -->
 <robot xmlns:xacro="https://ei.is.tuebingen.mpg.de/xacro">
-    <xacro:property name="material_name" value="material"/>
-    <xacro:property name="color" value="0.6 0.6 1.0"/>
-    <xacro:property name="opacity" value="1.0"/>
-    <xacro:macro name="add_geometry" params="origin_rpy origin_xyz mesh_file mesh_scale:='1'">
+    <xacro:macro name="add_geometry"
+        params="origin_rpy origin_xyz mesh_file material mesh_scale:='1'">
         <visual>
             <origin rpy="${origin_rpy}" xyz="${origin_xyz}"/>
@@ -11,7 +9,5 @@
                 <mesh scale="${mesh_scale} ${mesh_scale} ${mesh_scale}" filename="${mesh_file}"/>
             </geometry>
-            <material name="${material_name}">
-                <color rgba="${color} ${opacity}"/>
-            </material>
+            <material name="${material}" />
         </visual>
         <collision>
@@ -20,7 +16,4 @@
                 <mesh scale="${mesh_scale} ${mesh_scale} ${mesh_scale}" filename="${mesh_file}"/>
             </geometry>
-            <material name="${material_name}">
-                <color rgba="${color} ${opacity}"/>
-            </material>
         </collision>
     </xacro:macro>

File: xacro/stage.urdf.xacro (robot description, xacro)
@@ -2,4 +2,7 @@
 <robot name="stage" xmlns:xacro="https://ei.is.tuebingen.mpg.de/xacro">
     <xacro:include filename="macros.xacro" />
+    <material name="stage_material">
+        <color rgba="0.8 0.8 0.8 1.0" />
+    </material>
     <!-- Meshes -->
     <xacro:property name="mesh_file_extension" value="stl"/>
@@ -11,5 +14,6 @@
             origin_rpy="0 0 0"
             origin_xyz="0 0 0"
-            mesh_file="${stage_mesh}"/>
+            mesh_file="${stage_mesh}"
+            material="stage_material" />
         <xacro:add_inertia
             length_x="0.3"

File: xacro/trifinger.urdf.xacro (robot description, xacro)
@@ -20,8 +20,17 @@
         <origin xyz="0 0 0.34"/>
     </joint>
+    <material name="finger_0_material">
+        <color rgba="0.6 0.0 0.0 1.0" />
+    </material>
+    <material name="finger_120_material">
+        <color rgba="0.0 0.6 0.0 1.0" />
+    </material>
+    <material name="finger_240_material">
+        <color rgba="0.0 0.0 0.6 1.0" />
+    </material>
     <!-- Define the three fingers and place them relative to the upper holder -->
-    <xacro:finger suffix="_0"/>
-    <xacro:finger suffix="_120"/>
-    <xacro:finger suffix="_240"/>
+    <xacro:finger suffix="_0" material="finger_0_material" />
+    <xacro:finger suffix="_120" material="finger_120_material" />
+    <xacro:finger suffix="_240" material="finger_240_material" />
     <xacro:property name="offset" value="0.04"/> <!-- upper_holder to finger offset -->
     <xacro:property name="angle_0" value="${radians(0)}"/>

File: xacro/trifinger_with_stage.urdf.xacro (robot description, xacro)
@@ -9,4 +9,7 @@
     <xacro:property name="mesh_dir" value="package://robot_properties_manipulator/meshes/${mesh_file_extension}"/>
     <xacro:property name="stage_mesh" value="${mesh_dir}/BL-M_Table_ASM_big.${mesh_file_extension}"/>
+    <material name="stage_material">
+        <color rgba="0.8 0.8 0.8 1.0" />
+    </material>
     <link name="stage_link">
         <xacro:add_geometry
@@ -14,5 +17,6 @@
             origin_xyz="0 0 0"
             mesh_file="${stage_mesh}"
-            mesh_scale="1"/>
+            mesh_scale="1"
+            material="stage_material" />
         <xacro:add_inertia
             length_x="0.3"
