Commit message: added xacro for trifinger_without_stage

File: xacro/trifinger_with_stage.urdf.xacro (robot description, xacro)
@@ -2,8 +2,6 @@
 <robot name="finger_with_stage"
     xmlns:xacro="https://ei.is.tuebingen.mpg.de/xacro">
-    <xacro:include filename="finger_macro.urdf.xacro" />
+    <xacro:include filename="trifinger.urdf.xacro" />
     <xacro:include filename="macros.xacro" />
-    <!-- Define the global base_link and place all other objects relative to it. -->
-    <link name="base_link" />
     <!-- Adding the "stage" -->
     <!-- Meshes -->
@@ -28,33 +26,3 @@
         <origin xyz="0 0 0"/>
     </joint>
-    <!-- Define the upper holder -->
-    <link name="upper_holder_link" />
-    <joint name="stage_to_upper_holder_joint" type="fixed">
-        <parent link="stage_link"/>
-        <child link="upper_holder_link"/>
-        <origin xyz="0 0 0.34"/>
-    </joint>
-    <!-- Define the three fingers and place them relative to the upper holder -->
-    <xacro:finger suffix="_0"/>
-    <xacro:finger suffix="_120"/>
-    <xacro:finger suffix="_240"/>
-    <xacro:property name="offset" value="0.04"/> <!-- upper_holder to finger offset -->
-    <xacro:property name="angle_0" value="${radians(0)}"/>
-    <xacro:property name="angle_120" value="${radians(120)}"/>
-    <xacro:property name="angle_240" value="${radians(240)}"/>
-    <joint name="holder_to_finger_0" type="fixed">
-        <parent link="upper_holder_link"/>
-        <child link="finger_base_link_0"/>
-        <origin xyz="${offset * sin(angle_0)} ${offset * cos(angle_0)} 0" rpy="0 0 0"/>
-    </joint>
-    <joint name="holder_to_finger_120" type="fixed">
-        <parent link="upper_holder_link"/>
-        <child link="finger_base_link_120"/>
-        <origin xyz="${offset * sin(angle_120)} ${offset * cos(angle_120)} 0" rpy="0 0 -${angle_120}"/>
-    </joint>
-    <joint name="holder_to_finger_240" type="fixed">
-        <parent link="upper_holder_link"/>
-        <child link="finger_base_link_240"/>
-        <origin xyz="${offset * sin(angle_240)} ${offset * cos(angle_240)} 0" rpy="0 0 -${angle_240}"/>
-    </joint>
 </robot>

Commit message: Use high boundary in stage for TriFinger
Add a xacro file for the "TriFinger Stage" with the high boundary.
Boundary and table are kept in separate mesh files, so they can be
assigned different colours.

Use this in trifinger_stage.urdf.xacro.

File: xacro/trifinger_with_stage.urdf.xacro (robot description, xacro)
@@ -3,36 +3,4 @@
     xmlns:xacro="https://ei.is.tuebingen.mpg.de/xacro">
     <xacro:include filename="trifinger.urdf.xacro" />
-    <xacro:include filename="macros.xacro" />
-    <!-- Adding the "stage" -->
-    <!-- Meshes -->
-    <xacro:property name="mesh_file_extension" value="stl"/>
-    <xacro:property name="mesh_dir" value="package://robot_properties_fingers/meshes/${mesh_file_extension}"/>
-    <xacro:property name="stage_mesh" value="${mesh_dir}/BL-M_Table_ASM_big.${mesh_file_extension}"/>
-    <material name="stage_material">
-        <color rgba="0.8 0.8 0.8 1.0" />
-    </material>
-    <link name="stage_link">
-        <xacro:add_geometry
-            rpy="0 0 0"
-            xyz="0 0 0"
-            mesh_file="${stage_mesh}"
-            mesh_scale="1"
-            material="stage_material" />
-        <xacro:add_inertia
-            length_x="0.3"
-            length_y="0.3"
-            length_z="0.05"
-            mass="1"
-            com="0 0 0"/>
-            <!--
-            ROS uses meters for length. Since the new lower_link_mesh and the stage_mesh is made using millimeters as units,
-            scaling them down to 1/1000 of their current size loads them with the correct size.
-            -->
-    </link>
-    <!-- Define the stage -->
-    <joint name="base_to_stage" type="fixed">
-        <parent link="base_link"/>
-        <child link="stage_link"/>
-        <origin xyz="0 0 0"/>
-    </joint>
+    <xacro:include filename="trifinger_stage.urdf.xacro" />
 </robot>
