Commit message: added 3-finger urdf

File: xacro/finger_macro.urdf.xacro (robot description, xacro)
@@ -26,13 +26,18 @@
     <xacro:property name="centre_offset" value="0.014" />
     <xacro:property name="lower_link_mesh_scale" value="0.001 0.001 0.001" />
-    <xacro:property name="tip_padding" value="0" /> <!-- Flag for tip_padding. 0 = False -->
-    <xacro:property name="base_holder" value="0" /> <!-- Flag for upper base_holder. 0 = False -->
+    <xacro:property name="tip_padding" value="0" />
+    <xacro:property name="base_holder" value="0" />
+    <!--
+    Defining the "finger" macro which is used for both single and tri-finger.
+    The macro takes "idx" as a parameter for the three fingers.
+    In case of single finger, no "idx" value is passed.
+    -->
     <xacro:macro name="finger" params="idx:=''">
-        <!-- In case of single finger (i.e. when no idx is passed), we change the default values of the following. -->
+        <!-- In case of single finger (i.e. when no idx is passed), we change the default values of the following variables. -->
         <xacro:if value="${idx == ''}">
-            <xacro:property name="lower_link_mesh" value="${mesh_dir}/SIM_BL_FINGER_TIP_LINK.${mesh_file_extension}"/>
-            <xacro:property name="lower_link_mesh_scale" value="1 1 1" />
-            <xacro:property name="tip_padding" value="1" />
-            <xacro:property name="base_holder" value="1" />
+            <xacro:property name="lower_link_mesh" value="${mesh_dir}/SIM_BL_FINGER_TIP_LINK.${mesh_file_extension}"/> <!-- mesh for single finger -->
+            <xacro:property name="lower_link_mesh_scale" value="1 1 1" /> <!-- lower_link_mesh has different scale for single and 3-finger -->
+            <xacro:property name="tip_padding" value="1" /> <!-- Flag for tip_padding. 1 = True -->
+            <xacro:property name="base_holder" value="1" /> <!-- Flag for upper base_holder. 1 = True -->
         </xacro:if>
         <!--

Commit message: changed mesh scale for 3 fingers

File: xacro/finger_macro.urdf.xacro (robot description, xacro)
@@ -29,5 +29,5 @@
     scaling them down to 1/1000 of their current size loads them with the correct size.
     -->
-    <xacro:property name="lower_link_mesh_scale" value="0.001" />
+    <xacro:property name="lower_link_mesh_scale" value="1" />
     <xacro:property name="tip_padding" value="0" /> <!-- if this flag is set to 1 (True), finger padding is added at the finger tips -->
     <xacro:property name="base_holder" value="0" /> <!-- if this flag is set to 1 (True), an upper base_holder is added -->

File: xacro/trifinger_with_stage.urdf.xacro (robot description, xacro)
@@ -14,5 +14,5 @@
             origin_xyz="0 0 0"
             mesh_file="${stage_mesh}"
-            mesh_scale="0.001"/>
+            mesh_scale="1"/>
             <!--
             ROS uses meters for length. Since the new lower_link_mesh and the stage_mesh is made using millimeters as units,

Commit message: more 'realistic' inertias (manuel)

File: xacro/finger_macro.urdf.xacro (robot description, xacro)
@@ -38,5 +38,5 @@
     In case of single finger, no "suffix" value is passed.
     -->
-    <xacro:macro name="finger" params="suffix:=''">
+    <xacro:macro name="finger" params="material suffix:=''">
         <!-- In case of single finger (i.e. when no suffix is passed), we change the default values of the following variables. -->
         <xacro:if value="${suffix == ''}">
@@ -54,5 +54,6 @@
                 origin_rpy="0 0 0"
                 origin_xyz="0 ${upper_link_length} 0"
-                mesh_file="${upper_base_mesh}"/>
+                mesh_file="${upper_base_mesh}"
+                material="${material}" />
             <xacro:add_inertia
                 length_x="0.05"
@@ -67,5 +68,6 @@
                     origin_rpy="0 0 0"
                     origin_xyz="0 0 0"
-                    mesh_file="${base_holder_mesh}"/>
+                    mesh_file="${base_holder_mesh}"
+                    material="${material}" />
                 <!--
                   for some reason this link needs to have some inertia defined,
@@ -91,9 +93,10 @@
                 origin_rpy="0 0 0"
                 origin_xyz="0 -${upper_joint_center_offset} 0"
-                mesh_file="${upper_link_mesh}"/>
+                mesh_file="${upper_link_mesh}"
+                material="${material}" />
             <xacro:add_inertia
-                length_x="0.02"
+                length_x="0.04"
                 length_y="0.14"
-                length_z="0.02"
+                length_z="0.04"
                 mass="0.2"
                 com="0 0.06 0"/>
@@ -103,11 +106,12 @@
                 origin_rpy="${pi/2} 0 0"
                 origin_xyz="${mesh_x_offset} 0 0"
-                mesh_file="${middle_link_mesh}"/>
+                mesh_file="${middle_link_mesh}"
+                material="${material}" />
             <xacro:add_inertia
-                length_x="0.02"
-                length_y="0.02"
+                length_x="0.04"
+                length_y="0.04"
                 length_z="0.14"
                 mass="0.2"
-                com="${2 * mesh_x_offset} 0 -0.06"/>
+                com="${2 * mesh_x_offset} 0 -0.08"/>
         </link>
         <link name="finger_lower_link${suffix}">
@@ -116,17 +120,19 @@
                 origin_xyz="${mesh_x_offset} 0 0"
                 mesh_file="${lower_link_mesh}"
-                mesh_scale="${lower_link_mesh_scale}"/>
+                mesh_scale="${lower_link_mesh_scale}"
+                material="${material}" />
             <xacro:if value="${tip_padding == 1}"> <!-- tip_padding is added in case of single finger -->
                 <xacro:add_geometry
                     origin_rpy="0 0 0"
                     origin_xyz="0 0 -${lower_joint_to_tip_distance}"
-                    mesh_file="${tip_padding_mesh}"/>
+                    mesh_file="${tip_padding_mesh}"
+                    material="${material}" />
             </xacro:if>
             <xacro:add_inertia
-                length_x="0.01"
-                length_y="0.01"
+                length_x="0.02"
+                length_y="0.02"
                 length_z="0.14"
                 mass="0.05"
-                com="0 0 -0.07"/>
+                com="0 0 -0.06"/>
         </link>
         <!-- fixed link for finger tip -->

Commit message: Set weight of lower link to more realistic value
The weight of the lower link and tip was significantly over-estimated.
Set values that match more with the actual robot.

File: xacro/finger_macro.urdf.xacro (robot description, xacro)
@@ -32,5 +32,5 @@
     <xacro:property name="tip_padding" value="0" /> <!-- if this flag is set to 1 (True), finger padding is added at the finger tips -->
     <xacro:property name="base_holder" value="0" /> <!-- if this flag is set to 1 (True), an upper base_holder is added -->
-    <xacro:property name="tip_mass" value="0.075" />
+    <xacro:property name="tip_mass" value="0.02" />
     <!--
     Defining the "finger" macro which is used for both single and tri-finger.
@@ -45,5 +45,5 @@
             <xacro:property name="tip_padding" value="1" />
             <xacro:property name="base_holder" value="1" />
-            <xacro:property name="tip_mass" value="0.025" />
+            <xacro:property name="tip_mass" value="0.002" />
         </xacro:if>
         <!--
@@ -133,5 +133,5 @@
                 length_y="0.02"
                 length_z="0.14"
-                mass="0.05"
+                mass="0.01"
                 com="0 0 -0.06"/>
         </link>

Commit message: Use lower link of single finger for trifinger
As the TriFinger has now more ball-shaped tips, the actual shape matches
more the mesh of the single finger.  Therefore use the same lower link
mesh on both robots until we have a more accurate one for the TriFinger.

File: xacro/finger_macro.urdf.xacro (robot description, xacro)
@@ -16,5 +16,8 @@
     <xacro:property name="upper_link_mesh" value="${mesh_dir}/SIM__BL-Finger_Proximal.${mesh_file_extension}"/>
     <xacro:property name="middle_link_mesh" value="${mesh_dir}/SIM__BL-Finger_Intermediate.${mesh_file_extension}"/>
-    <xacro:property name="lower_link_mesh" value="${mesh_dir}/Tip_link_Modular_SIM.${mesh_file_extension}"/>
+    <!-- <xacro:property name="lower_link_mesh" value="${mesh_dir}/Tip_link_Modular_SIM.${mesh_file_extension}"/> -->
+    <!-- With the round tip the lower link is closer to the one of the single finger.
+         TODO: set a proper mesh matching the actual link of the TriFinger. -->
+    <xacro:property name="lower_link_mesh" value="${mesh_dir}/SIM_BL_FINGER_TIP_LINK.${mesh_file_extension}"/>
     <xacro:property name="tip_padding_mesh" value="${mesh_dir}/finger_padding.${mesh_file_extension}"/>
     <!-- Distance from outer edge of the link to the joint center -->

Commit message: Limit the lower joint to the negative range
This way the "knee" is always pointing away from the centre and thus
collisions between the fingers are reduced.

File: xacro/finger_macro.urdf.xacro (robot description, xacro)
@@ -172,5 +172,6 @@
             <parent link="finger_middle_link${suffix}"/>
             <child link="finger_lower_link${suffix}"/>
-            <limit effort="1000" lower="${radians(-172)}" upper="${radians(172)}" velocity="1000"/>
+            <!-- <limit effort="1000" lower="${radians(-172)}" upper="${radians(172)}" velocity="1000"/> -->
+            <limit effort="1000" lower="${radians(-172)}" upper="${radians(-2)}" velocity="1000"/>
             <axis xyz="1 0 0"/>
             <origin rpy="0 0 0" xyz="0 0 -${middle_to_lower_joint_distance}"/>

Commit message: Rename package to robot_properties_fingers

File: xacro/finger_macro.urdf.xacro (robot description, xacro)
@@ -11,5 +11,5 @@
     <!-- Meshes -->
     <xacro:property name="mesh_file_extension" value="stl"/>
-    <xacro:property name="mesh_dir" value="package://robot_properties_manipulator/meshes/${mesh_file_extension}"/>
+    <xacro:property name="mesh_dir" value="package://robot_properties_fingers/meshes/${mesh_file_extension}"/>
     <xacro:property name="upper_base_mesh" value="${mesh_dir}/SIM__BL-Finger_Base.${mesh_file_extension}"/>
     <xacro:property name="base_holder_mesh" value="${mesh_dir}/BL_Finger_Holder_SIM.${mesh_file_extension}"/>

File: xacro/stage.urdf.xacro (robot description, xacro)
@@ -7,5 +7,5 @@
     <!-- Meshes -->
     <xacro:property name="mesh_file_extension" value="stl"/>
-    <xacro:property name="mesh_dir" value="package://robot_properties_manipulator/meshes/${mesh_file_extension}"/>
+    <xacro:property name="mesh_dir" value="package://robot_properties_fingers/meshes/${mesh_file_extension}"/>
     <xacro:property name="stage_mesh" value="${mesh_dir}/Stage_simplified.${mesh_file_extension}"/>
     <!-- add the "stage" -->

File: xacro/trifinger_with_stage.urdf.xacro (robot description, xacro)
@@ -7,5 +7,5 @@
     <!-- Meshes -->
     <xacro:property name="mesh_file_extension" value="stl"/>
-    <xacro:property name="mesh_dir" value="package://robot_properties_manipulator/meshes/${mesh_file_extension}"/>
+    <xacro:property name="mesh_dir" value="package://robot_properties_fingers/meshes/${mesh_file_extension}"/>
     <xacro:property name="stage_mesh" value="${mesh_dir}/BL-M_Table_ASM_big.${mesh_file_extension}"/>
     <material name="stage_material">

Commit message: {origin_xyz -> xyz}, {origin_rpy -> rpy} in the add geometry tags

File: xacro/finger_macro.urdf.xacro (robot description, xacro)
@@ -55,6 +55,6 @@
         <link name="finger_base_link${suffix}">
             <xacro:add_geometry
-                origin_rpy="0 0 0"
-                origin_xyz="0 ${upper_link_length} 0"
+                rpy="0 0 0"
+                xyz="0 ${upper_link_length} 0"
                 mesh_file="${upper_base_mesh}"
                 material="${material}" />
@@ -69,6 +69,6 @@
             <link name="finger_upper_holder_link${suffix}">
                 <xacro:add_geometry
-                    origin_rpy="0 0 0"
-                    origin_xyz="0 0 0"
+                    rpy="0 0 0"
+                    xyz="0 0 0"
                     mesh_file="${base_holder_mesh}"
                     material="${material}" />
@@ -94,6 +94,6 @@
         <link name="finger_upper_link${suffix}">
             <xacro:add_geometry
-                origin_rpy="0 0 0"
-                origin_xyz="0 -${upper_joint_center_offset} 0"
+                rpy="0 0 0"
+                xyz="0 -${upper_joint_center_offset} 0"
                 mesh_file="${upper_link_mesh}"
                 material="${material}" />
@@ -107,6 +107,6 @@
         <link name="finger_middle_link${suffix}">
             <xacro:add_geometry
-                origin_rpy="${pi/2} 0 0"
-                origin_xyz="${mesh_x_offset} 0 0"
+                rpy="${pi/2} 0 0"
+                xyz="${mesh_x_offset} 0 0"
                 mesh_file="${middle_link_mesh}"
                 material="${material}" />
@@ -120,6 +120,6 @@
         <link name="finger_lower_link${suffix}">
             <xacro:add_geometry
-                origin_rpy="${pi/2} 0 0"
-                origin_xyz="${mesh_x_offset} 0 0"
+                rpy="${pi/2} 0 0"
+                xyz="${mesh_x_offset} 0 0"
                 mesh_file="${lower_link_mesh}"
                 mesh_scale="${lower_link_mesh_scale}"
@@ -127,6 +127,6 @@
             <xacro:if value="${tip_padding == 1}"> <!-- tip_padding is added in case of single finger -->
                 <xacro:add_geometry
-                    origin_rpy="0 0 0"
-                    origin_xyz="0 0 -${lower_joint_to_tip_distance}"
+                    rpy="0 0 0"
+                    xyz="0 0 -${lower_joint_to_tip_distance}"
                     mesh_file="${tip_padding_mesh}"
                     material="${material}" />

File: xacro/macros.xacro (robot description, xacro)
@@ -3,7 +3,7 @@
 <robot xmlns:xacro="https://ei.is.tuebingen.mpg.de/xacro">
     <xacro:macro name="add_geometry"
-        params="origin_rpy origin_xyz mesh_file material mesh_scale:='1'">
+        params="rpy xyz mesh_file material mesh_scale:='1'">
         <visual>
-            <origin rpy="${origin_rpy}" xyz="${origin_xyz}"/>
+            <origin rpy="${rpy}" xyz="${xyz}"/>
             <geometry>
                 <mesh scale="${mesh_scale} ${mesh_scale} ${mesh_scale}" filename="${mesh_file}"/>
@@ -12,5 +12,5 @@
         </visual>
         <collision>
-            <origin rpy="${origin_rpy}" xyz="${origin_xyz}"/>
+            <origin rpy="${rpy}" xyz="${xyz}"/>
             <geometry>
                 <mesh scale="${mesh_scale} ${mesh_scale} ${mesh_scale}" filename="${mesh_file}"/>

File: xacro/stage.urdf.xacro (robot description, xacro)
@@ -12,6 +12,6 @@
     <link name="stage_link">
         <xacro:add_geometry
-            origin_rpy="0 0 0"
-            origin_xyz="0 0 0"
+            rpy="0 0 0"
+            xyz="0 0 0"
             mesh_file="${stage_mesh}"
             material="stage_material" />

File: xacro/trifinger_with_stage.urdf.xacro (robot description, xacro)
@@ -14,6 +14,6 @@
     <link name="stage_link">
         <xacro:add_geometry
-            origin_rpy="0 0 0"
-            origin_xyz="0 0 0"
+            rpy="0 0 0"
+            xyz="0 0 0"
             mesh_file="${stage_mesh}"
             mesh_scale="1"

Commit message: Set back to the original joint range for the lower joint

File: xacro/finger_macro.urdf.xacro (robot description, xacro)
@@ -175,6 +175,5 @@
             <parent link="finger_middle_link${suffix}"/>
             <child link="finger_lower_link${suffix}"/>
-            <!-- <limit effort="1000" lower="${radians(-172)}" upper="${radians(172)}" velocity="1000"/> -->
-            <limit effort="1000" lower="${radians(-172)}" upper="${radians(-2)}" velocity="1000"/>
+            <limit effort="1000" lower="${radians(-172)}" upper="${radians(172)}" velocity="1000"/>
             <axis xyz="1 0 0"/>
             <origin rpy="0 0 0" xyz="0 0 -${middle_to_lower_joint_distance}"/>
