Commit message: fixed meshes to avoid self-collision

File: xacro/macros.xacro (robot description, xacro)
@@ -18,5 +18,5 @@
             <origin rpy="${origin_rpy}" xyz="${origin_xyz}"/>
             <geometry>
-                <mesh filename="${mesh_file}"/>
+                <mesh scale="${mesh_scale} ${mesh_scale} ${mesh_scale}" filename="${mesh_file}"/>
             </geometry>
             <material name="${material_name}">

Commit message: Remove collision geometry of center holder
The fingers were colliding with the center holder part.  As the fingers
anyway cannot physically reach there, simply remove the collision
geometry from that link (i.e. use only a visual one).

File: xacro/macros.xacro (robot description, xacro)
@@ -18,4 +18,14 @@
         </collision>
     </xacro:macro>
+    <xacro:macro name="add_visual_geometry"
+        params="rpy xyz mesh_file material mesh_scale:='1'">
+        <visual>
+            <origin rpy="${rpy}" xyz="${xyz}"/>
+            <geometry>
+                <mesh scale="${mesh_scale} ${mesh_scale} ${mesh_scale}" filename="${mesh_file}"/>
+            </geometry>
+            <material name="${material}" />
+        </visual>
+    </xacro:macro>
     <xacro:macro name="add_inertia" params="length_x length_y length_z mass com">
         <inertial>

File: xacro/pro/trifingerpro.urdf.xacro (robot description, xacro)
@@ -16,11 +16,11 @@
     <!-- Define the upper holder -->
     <link name="upper_holder_link">
+        <xacro:add_visual_geometry
+            rpy="0 0 0"
+            xyz="0 0 0"
+            mesh_file="${center_link_mesh}"
+            material="finger_material"
+            mesh_scale="1." />
         <!-- add inertial to suppress warning -->
-        <xacro:add_geometry
-                        rpy="0 0 0"
-                        xyz="0 0 0"
-                        mesh_file="${center_link_mesh}"
-                        material="finger_material"
-                        mesh_scale="1." />
         <xacro:add_inertia
             length_x="0.005"
