Commit message: Add inertia to upper_holder_link to suppress warning
This is a static link that does not move, so the ineria of it does not
matter.  However, we need to add inertia values to _each_ joint,
otherwise bullet will print a warning.

File: xacro/trifinger.urdf.xacro (robot description, xacro)
@@ -6,13 +6,22 @@
     <!-- Define the global base_link and place all other objects relative to it. -->
     <link name="base_link">
-      <xacro:add_inertia
-          length_x="0.005"
-          length_y="0.005"
-          length_z="0.005"
-          mass="1"
-          com="0 0 0"/>
+        <!-- add inertial to suppress warning -->
+        <xacro:add_inertia
+            length_x="0.005"
+            length_y="0.005"
+            length_z="0.005"
+            mass="1"
+            com="0 0 0"/>
     </link>
     <!-- Define the upper holder -->
-    <link name="upper_holder_link" />
+    <link name="upper_holder_link">
+        <!-- add inertial to suppress warning -->
+        <xacro:add_inertia
+            length_x="0.005"
+            length_y="0.005"
+            length_z="0.005"
+            mass="1"
+            com="0 0 0"/>
+    </link>
     <joint name="base_to_upper_holder_joint" type="fixed">
         <parent link="base_link"/>

Commit message: Set height of TriFingerOne to 29 cm
This is currently the height of the real robot when the table is mounted
on the lowest level.

File: xacro/trifinger.urdf.xacro (robot description, xacro)
@@ -27,5 +27,5 @@
         <parent link="base_link"/>
         <child link="upper_holder_link"/>
-        <origin xyz="0 0 0.34"/>
+        <origin xyz="0 0 0.29"/>
     </joint>
     <material name="finger_0_material">
