Commit message: Remove "edu" from link/joint names of (Tri)FingerEdu
Just keep "finger_" as prefix for link and joint names.  This way, the
different versions of the fingers use the same names which makes it
easier to exchange them, for example in the simulation.

File: xacro/edu/fingeredu.urdf.xacro (robot description, xacro)
@@ -32,5 +32,5 @@
     <joint name="base_to_finger" type="fixed">
         <parent link="base_link"/>
-        <child link="fingeredu_base_link"/>
+        <child link="finger_base_link"/>
         <origin xyz="0 0 ${distance_to_ground}"/>
     </joint>

File: xacro/edu/fingeredu_macro.xacro (robot description, xacro)
@@ -23,5 +23,5 @@
         Fixed links for the finger base (parts where the upper link is mounted).
         -->
-        <link name="fingeredu_base_link${suffix}">
+        <link name="finger_base_link${suffix}">
             <xacro:add_geometry
                 rpy="0 0 0"
@@ -61,5 +61,5 @@
         <!-- The movable links (upper, middle and lower) of the finger. -->
         <!-- FIXME inertias are not correct! -->
-        <link name="fingeredu_upper_link${suffix}">
+        <link name="finger_upper_link${suffix}">
             <xacro:add_geometry
                 rpy="0 0 0"
@@ -78,5 +78,5 @@
             </inertial>
         </link>
-        <link name="fingeredu_middle_link${suffix}">
+        <link name="finger_middle_link${suffix}">
             <xacro:add_geometry
                 rpy="0 0 0"
@@ -92,5 +92,5 @@
             </inertial>
         </link>
-        <link name="fingeredu_lower_link${suffix}">
+        <link name="finger_lower_link${suffix}">
             <xacro:add_geometry
                 rpy="0 0 0"
@@ -110,5 +110,5 @@
         </link>
         <!-- fixed link for finger tip -->
-        <link name="fingeredu_tip_link${suffix}">
+        <link name="finger_tip_link${suffix}">
             <!-- TODO: Inertia of tip is just a very rough estimate -->
             <xacro:add_inertia
@@ -119,27 +119,27 @@
                 mass="0.01"/>
         </link>
-        <joint name="fingeredu_lower_to_tip_joint${suffix}" type="fixed">
-            <parent link="fingeredu_lower_link${suffix}"/>
-            <child link="fingeredu_tip_link${suffix}"/>
+        <joint name="finger_lower_to_tip_joint${suffix}" type="fixed">
+            <parent link="finger_lower_link${suffix}"/>
+            <child link="finger_tip_link${suffix}"/>
             <origin xyz="0 -0.008 -0.16"/>
         </joint>
         <!-- kinematics -->
-        <joint name="fingeredu_base_to_upper_joint${suffix}" type="revolute">
-            <parent link="fingeredu_base_link${suffix}"/>
-            <child link="fingeredu_upper_link${suffix}"/>
+        <joint name="finger_base_to_upper_joint${suffix}" type="revolute">
+            <parent link="finger_base_link${suffix}"/>
+            <child link="finger_upper_link${suffix}"/>
             <limit effort="1000" lower="-${pi/2}" upper="${pi/2}" velocity="1000"/>
             <axis xyz="-1 0 0"/>
             <origin rpy="0 0 0" xyz="0 0 0"/>
         </joint>
-        <joint name="fingeredu_upper_to_middle_joint${suffix}" type="revolute">
-            <parent link="fingeredu_upper_link${suffix}"/>
-            <child link="fingeredu_middle_link${suffix}"/>
+        <joint name="finger_upper_to_middle_joint${suffix}" type="revolute">
+            <parent link="finger_upper_link${suffix}"/>
+            <child link="finger_middle_link${suffix}"/>
             <limit effort="1000" lower="-${pi/2}" upper="${pi/2}" velocity="1000"/>
             <axis xyz="0 1 0"/>
             <origin rpy="0 0 0" xyz="0 -0.014 0"/>
         </joint>
-        <joint name="fingeredu_middle_to_lower_joint${suffix}" type="revolute">
-            <parent link="fingeredu_middle_link${suffix}"/>
-            <child link="fingeredu_lower_link${suffix}"/>
+        <joint name="finger_middle_to_lower_joint${suffix}" type="revolute">
+            <parent link="finger_middle_link${suffix}"/>
+            <child link="finger_lower_link${suffix}"/>
             <limit effort="1000" lower="-${pi}" upper="${pi}" velocity="1000"/>
             <axis xyz="0 1 0"/>

File: xacro/edu/trifingeredu.urdf.xacro (robot description, xacro)
@@ -19,8 +19,8 @@
     </link>
     <!-- Define the upper holder -->
-    <link name="trifingeredu_base_link" />
-    <joint name="base_to_trifingeredu_base_joint" type="fixed">
+    <link name="trifinger_base_link" />
+    <joint name="base_to_trifinger_base_joint" type="fixed">
         <parent link="base_link"/>
-        <child link="trifingeredu_base_link"/>
+        <child link="trifinger_base_link"/>
         <origin xyz="0 0 ${distance_to_ground}"/>
     </joint>
@@ -38,17 +38,17 @@
     <xacro:fingeredu suffix="_120" material="fingeredu_120_material" />
     <xacro:fingeredu suffix="_240" material="fingeredu_240_material" />
-    <joint name="base_to_fingeredu_0" type="fixed">
-        <parent link="trifingeredu_base_link"/>
-        <child link="fingeredu_base_link_0"/>
+    <joint name="base_to_finger_0" type="fixed">
+        <parent link="trifinger_base_link"/>
+        <child link="finger_base_link_0"/>
         <origin xyz="${distance_to_center * cos(-angle_0)} ${distance_to_center * sin(-angle_0)} 0" rpy="0 0 0"/>
     </joint>
-    <joint name="base_to_fingeredu_120" type="fixed">
-        <parent link="trifingeredu_base_link"/>
-        <child link="fingeredu_base_link_120"/>
+    <joint name="base_to_finger_120" type="fixed">
+        <parent link="trifinger_base_link"/>
+        <child link="finger_base_link_120"/>
         <origin xyz="${distance_to_center * cos(-angle_120)} ${distance_to_center * sin(-angle_120)} 0" rpy="0 0 -${angle_120}"/>
     </joint>
-    <joint name="base_to_fingeredu_240" type="fixed">
-        <parent link="trifingeredu_base_link"/>
-        <child link="fingeredu_base_link_240"/>
+    <joint name="base_to_finger_240" type="fixed">
+        <parent link="trifinger_base_link"/>
+        <child link="finger_base_link_240"/>
         <origin xyz="${distance_to_center * cos(-angle_240)} ${distance_to_center * sin(-angle_240)} 0" rpy="0 0 -${angle_240}"/>
     </joint>
