Commit message: Use same orientation of world frame in TriFingerOne and Edu
Rotate the world frame such that the axes go in the same direction for
TriFingerOne and TriFingerEdu.

File: xacro/edu/trifingeredu.urdf.xacro (robot description, xacro)
@@ -23,5 +23,5 @@
         <parent link="base_link"/>
         <child link="trifinger_base_link"/>
-        <origin xyz="0 0 ${distance_to_ground}"/>
+        <origin xyz="0 0 ${distance_to_ground}" rpy="0 0 ${radians(-90)}" />
     </joint>
     <material name="fingeredu_0_material">

Commit message: Add inertial to fixed frame to suppress warning

File: xacro/edu/trifingeredu.urdf.xacro (robot description, xacro)
@@ -19,5 +19,13 @@
     </link>
     <!-- Define the upper holder -->
-    <link name="trifinger_base_link" />
+    <link name="trifinger_base_link">
+        <!-- add inertial to suppress warning -->
+        <xacro:add_inertia
+            length_x="0.005"
+            length_y="0.005"
+            length_z="0.005"
+            mass="1"
+            com="0 0 0"/>
+    </link>
     <joint name="base_to_trifinger_base_joint" type="fixed">
         <parent link="base_link"/>
