Commit message: Add finger tip link (estimated position)

File: xacro/pro/fingerpro_macro.xacro (robot description, xacro)
@@ -26,4 +26,6 @@
     <xacro:property name="center_offset" value="0.0235" />
     <xacro:property name="mesh_x_offset" value="0.014" />
+    <xacro:property name="lower_joint_to_tip_distance" value="0.16" />
+    <xacro:property name="tip_mass" value="0.02" />
     <!--
     Defining the "finger" macro which is used for both single and tri-finger.
@@ -92,9 +94,20 @@
                 com="0 0 -0.06"/>
         </link>
+        <!-- fixed link for finger tip -->
+        <link name="finger_tip_link${suffix}">
+            <xacro:add_inertia
+                length_x="0.01"
+                length_y="0.01"
+                length_z="0.01"
+                com="0 0 0"
+                mass="${tip_mass}"/>
+        </link>
+        <joint name="finger_lower_to_tip_joint${suffix}" type="fixed">
+            <parent link="finger_lower_link${suffix}"/>
+            <child link="finger_tip_link${suffix}"/>
+            <origin xyz="0.0185 0 -${lower_joint_to_tip_distance}"/>
+        </joint>
         <!-- kinematics -->
-        <!-- TODO: joint limits are based on values from wiki
-        (https://atlas.is.localnet/confluence/display/AMDW/Forward+Kinematics) but
-        should be verified on the real system (especially the finger tip limits look
-        a bit too big when visualizing the model. -->
+        <!-- FIXME: Set proper joint limits -->
         <joint name="finger_base_to_upper_joint${suffix}" type="revolute">
             <parent link="finger_base_link${suffix}"/>

Commit message: Set joint limits according to robot configuration

File: xacro/pro/fingerpro_macro.xacro (robot description, xacro)
@@ -109,9 +109,11 @@
         </joint>
         <!-- kinematics -->
-        <!-- FIXME: Set proper joint limits -->
+        <!-- NOTE: Joint limits are set according to soft limits in the
+             configuration of the real robot (i.e. not according to physical
+             limits). -->
         <joint name="finger_base_to_upper_joint${suffix}" type="revolute">
             <parent link="finger_base_link${suffix}"/>
             <child link="finger_upper_link${suffix}"/>
-            <limit effort="1000" lower="-${pi/2}" upper="${pi/2}" velocity="1000"/>
+            <limit effort="1000" lower="-0.9" upper="1.4" velocity="1000"/>
             <axis xyz="0 1 0"/>
             <origin rpy="0 0 0" xyz="0 0 0"/>
@@ -120,5 +122,5 @@
             <parent link="finger_upper_link${suffix}"/>
             <child link="finger_middle_link${suffix}"/>
-            <limit effort="1000" lower="${radians(-77.5)}" upper="${radians(257.5)}" velocity="1000"/>
+            <limit effort="1000" lower="-1.57" upper="1.57" velocity="1000"/>
             <axis xyz="1 0 0"/>
             <origin rpy="0 0 0" xyz="${middle_dx} ${middle_dy+center_offset} 0"/>
@@ -127,5 +129,5 @@
             <parent link="finger_middle_link${suffix}"/>
             <child link="finger_lower_link${suffix}"/>
-            <limit effort="1000" lower="${radians(-172)}" upper="${radians(172)}" velocity="1000"/>
+            <limit effort="1000" lower="-2.7" upper="2.7" velocity="1000"/>
             <axis xyz="1 0 0"/>
             <origin rpy="0 0 0" xyz="${lower_dx} 0 -${lower_dy}"/>

Commit message: adds new mesh and modifies xacro macro for tip

File: xacro/pro/fingerpro_macro.xacro (robot description, xacro)
@@ -26,5 +26,5 @@
     <xacro:property name="center_offset" value="0.0235" />
     <xacro:property name="mesh_x_offset" value="0.014" />
-    <xacro:property name="lower_joint_to_tip_distance" value="0.16" />
+    <xacro:property name="lower_joint_to_tip_distance" value="0.1626" />
     <xacro:property name="tip_mass" value="0.02" />
     <!--

File: xacro/pro/trifingerpro.urdf.xacro (robot description, xacro)
@@ -33,5 +33,5 @@
         <parent link="base_link"/>
         <child link="upper_holder_link"/>
-        <origin xyz="0 0 0.29"/>
+        <origin xyz="0 0 0.34"/>
     </joint>
     <material name="finger_0_material">

Commit message: Set mass of tip link to zero
This is just a logical link so we can easily refer to the tip of the
finger.  Physically it is part of the lower link, so there is no extra
mass to add.

File: xacro/pro/fingerpro_macro.xacro (robot description, xacro)
@@ -27,5 +27,4 @@
     <xacro:property name="mesh_x_offset" value="0.014" />
     <xacro:property name="lower_joint_to_tip_distance" value="0.1626" />
-    <xacro:property name="tip_mass" value="0.02" />
     <!--
     Defining the "finger" macro which is used for both single and tri-finger.
@@ -101,5 +100,5 @@
                 length_z="0.01"
                 com="0 0 0"
-                mass="${tip_mass}"/>
+                mass="0"/>
         </link>
         <joint name="finger_lower_to_tip_joint${suffix}" type="fixed">

Commit message: Set lower joint upper limit to zero
Only allow this joint to move in one direction.  This prevents states
where the robot can easily get stuck and should not be a serious
limitation for the intended manipulation tasks.

Further it has the side effect that the inverse kinematics only has one
solution for most positions.

File: xacro/pro/fingerpro_macro.xacro (robot description, xacro)
@@ -128,5 +128,5 @@
             <parent link="finger_middle_link${suffix}"/>
             <child link="finger_lower_link${suffix}"/>
-            <limit effort="1000" lower="-2.7" upper="2.7" velocity="1000"/>
+            <limit effort="1000" lower="-2.7" upper="0.0" velocity="1000"/>
             <axis xyz="1 0 0"/>
             <origin rpy="0 0 0" xyz="${lower_dx} 0 -${lower_dy}"/>

Commit message: Use the split mesh for lower and tip link

File: xacro/pro/fingerpro_macro.xacro (robot description, xacro)
@@ -16,5 +16,6 @@
     <xacro:property name="upper_link_mesh" value="${mesh_dir}/SIM__BL-Finger_Proximal.${mesh_file_extension}"/>
     <xacro:property name="middle_link_mesh" value="${mesh_dir}/SIM__BL-Finger_Intermediate.${mesh_file_extension}"/>
-    <xacro:property name="lower_link_mesh" value="${mesh_dir}/SIM__BL-Finger_Tip.${mesh_file_extension}"/>
+    <xacro:property name="lower_link_mesh" value="${mesh_dir}/SIM__BL-Finger_Tip_without_tip.${mesh_file_extension}"/>
+    <xacro:property name="tip_link_mesh" value="${mesh_dir}/SIM__BL-Finger_Tip_actual_tip.${mesh_file_extension}"/>
     <!-- Distance from outer edge of the link to the joint center -->
     <xacro:property name="upper_link_length" value="0.20945" />
@@ -95,4 +96,10 @@
         <!-- fixed link for finger tip -->
         <link name="finger_tip_link${suffix}">
+            <xacro:add_geometry
+                rpy="${pi/2} 0 0"
+                xyz="-0.0185 0 ${lower_joint_to_tip_distance}"
+                mesh_file="${tip_link_mesh}"
+                material="${material}"
+                mesh_scale="1."/>
             <xacro:add_inertia
                 length_x="0.01"

Commit message: Set joint limits of TriFingerPro as on the real robot

File: xacro/pro/fingerpro_macro.xacro (robot description, xacro)
@@ -121,5 +121,5 @@
             <parent link="finger_base_link${suffix}"/>
             <child link="finger_upper_link${suffix}"/>
-            <limit effort="1000" lower="-0.9" upper="1.4" velocity="1000"/>
+            <limit effort="1000" lower="-0.33" upper="1.0" velocity="1000"/>
             <axis xyz="0 1 0"/>
             <origin rpy="0 0 0" xyz="0 0 0"/>
@@ -128,5 +128,5 @@
             <parent link="finger_upper_link${suffix}"/>
             <child link="finger_middle_link${suffix}"/>
-            <limit effort="1000" lower="-1.57" upper="1.57" velocity="1000"/>
+            <limit effort="1000" lower="0.0" upper="1.57" velocity="1000"/>
             <axis xyz="1 0 0"/>
             <origin rpy="0 0 0" xyz="${middle_dx} ${middle_dy+center_offset} 0"/>

Commit message: Add black parts (motor, cables, ...) of TriFingerPro
Since pyBullet doesn't support visuals with different materials on the
same link, add the black parts as separate fixed links.

File: xacro/pro/fingerpro_macro.xacro (robot description, xacro)
@@ -18,4 +18,5 @@
     <xacro:property name="lower_link_mesh" value="${mesh_dir}/SIM__BL-Finger_Tip_without_tip.${mesh_file_extension}"/>
     <xacro:property name="tip_link_mesh" value="${mesh_dir}/SIM__BL-Finger_Tip_actual_tip.${mesh_file_extension}"/>
+    <xacro:property name="motor_mesh" value="${mesh_dir}/SIM__BL-Finger_Motor.stl"/>
     <!-- Distance from outer edge of the link to the joint center -->
     <xacro:property name="upper_link_length" value="0.20945" />
@@ -28,4 +29,10 @@
     <xacro:property name="mesh_x_offset" value="0.014" />
     <xacro:property name="lower_joint_to_tip_distance" value="0.1626" />
+    <material name="fingerpro_shell">
+        <color rgba="0.83 0.79 0.82 1.0" />
+    </material>
+    <material name="fingerpro_motor">
+        <color rgba="0.17 0.17 0.17 1.0" />
+    </material>
     <!--
     Defining the "finger" macro which is used for both single and tri-finger.
@@ -33,5 +40,5 @@
     In case of single finger, no "suffix" value is passed.
     -->
-    <xacro:macro name="fingerpro" params="material suffix:=''">
+    <xacro:macro name="fingerpro" params="suffix:=''">
         <!--
         Fixed links for the finger base (parts where the upper link is mounted).
@@ -43,5 +50,5 @@
                 xyz="0 ${upper_link_length+center_offset} 0"
                 mesh_file="${upper_base_mesh}"
-                material="${material}"
+                material="fingerpro_shell"
                 mesh_scale="1." />
             <xacro:add_inertia
@@ -57,5 +64,5 @@
                 xyz="0 ${center_offset} 0"
                 mesh_file="${upper_link_mesh}"
-                material="${material}"
+                material="fingerpro_shell"
                 mesh_scale="1." />
             <xacro:add_inertia
@@ -66,4 +73,43 @@
                 com="0 0.06 0"/>
         </link>
+        <link name="finger_upper_link_motor${suffix}">
+            <!-- motor -->
+            <visual>
+                <origin xyz="0.018 0.141 -0.001" />
+                <geometry>
+                    <mesh filename="${motor_mesh}"/>
+                </geometry>
+                <material name="fingerpro_motor" />
+            </visual>
+            <!-- end stop -->
+            <visual>
+                <origin xyz="0.015 0.06 0" rpy="0 ${pi/2} 0" />
+                <geometry>
+                    <cylinder length="0.015" radius="0.005"/>
+                </geometry>
+                <material name="fingerpro_motor" />
+            </visual>
+            <!-- cables -->
+            <visual>
+                <origin xyz="-0.008 0.1 0" rpy="${pi/2} 0 0" />
+                <geometry>
+                    <cylinder length="0.12" radius="0.002"/>
+                </geometry>
+                <material name="fingerpro_motor" />
+            </visual>
+            <!-- opening on lower joint -->
+            <visual>
+                <origin xyz="-0.008 0.026 0" rpy="0 ${pi/2} 0" />
+                <geometry>
+                    <cylinder length="0.002" radius="0.014"/>
+                </geometry>
+                <material name="fingerpro_motor" />
+            </visual>
+        </link>
+        <joint name="finger_upper_to_motor_joint${suffix}" type="fixed">
+            <parent link="finger_upper_link${suffix}"/>
+            <child link="finger_upper_link_motor${suffix}"/>
+            <origin xyz="0 ${center_offset} 0" />
+        </joint>
         <link name="finger_middle_link${suffix}">
             <xacro:add_geometry
@@ -71,5 +117,5 @@
                 xyz="0 0 0"
                 mesh_file="${middle_link_mesh}"
-                material="${material}"
+                material="fingerpro_shell"
                 mesh_scale="1." />
             <xacro:add_inertia
@@ -80,4 +126,42 @@
                 com="${2 * mesh_x_offset} 0 -0.08"/>
         </link>
+        <link name="finger_middle_link_motor${suffix}">
+            <!-- motor -->
+            <visual>
+                <origin xyz="0.048 0 -0.046" />
+                <geometry>
+                    <mesh filename="${motor_mesh}"/>
+                </geometry>
+                <material name="fingerpro_motor" />
+            </visual>
+            <!-- end stop -->
+            <visual>
+                <origin xyz="0.048 0 -0.13" rpy="0 ${pi/2} 0" />
+                <geometry>
+                    <cylinder length="0.015" radius="0.005"/>
+                </geometry>
+                <material name="fingerpro_motor" />
+            </visual>
+            <!-- cables -->
+            <visual>
+                <origin xyz="0.025 0 -0.09" />
+                <geometry>
+                    <cylinder length="0.12" radius="0.002"/>
+                </geometry>
+                <material name="fingerpro_motor" />
+            </visual>
+            <!-- opening on lower joint -->
+            <visual>
+                <origin xyz="0.024 0 -0.16" rpy="0 ${pi/2} 0" />
+                <geometry>
+                    <cylinder length="0.002" radius="0.014"/>
+                </geometry>
+                <material name="fingerpro_motor" />
+            </visual>
+        </link>
+        <joint name="finger_middle_to_motor_joint${suffix}" type="fixed">
+            <parent link="finger_middle_link${suffix}"/>
+            <child link="finger_middle_link_motor${suffix}"/>
+        </joint>
         <link name="finger_lower_link${suffix}">
             <xacro:add_geometry
@@ -85,5 +169,5 @@
                 xyz="0 0 0"
                 mesh_file="${lower_link_mesh}"
-                material="${material}"
+                material="fingerpro_shell"
                 mesh_scale="1."/>
             <xacro:add_inertia
@@ -100,5 +184,5 @@
                 xyz="-0.0185 0 ${lower_joint_to_tip_distance}"
                 mesh_file="${tip_link_mesh}"
-                material="${material}"
+                material="fingerpro_shell"
                 mesh_scale="1."/>
             <xacro:add_inertia

Commit message: More realistic colours for FingerPro

File: xacro/pro/fingerpro_macro.xacro (robot description, xacro)
@@ -30,5 +30,10 @@
     <xacro:property name="lower_joint_to_tip_distance" value="0.1626" />
     <material name="fingerpro_shell">
-        <color rgba="0.83 0.79 0.82 1.0" />
+        <!-- colour from image -->
+        <color rgba="0.804 0.764 0.761 1.0" />
+    </material>
+    <material name="fingerpro_tip">
+        <!-- colour from image -->
+        <color rgba="0.33 0.36 0.37 1.0" />
     </material>
     <material name="fingerpro_motor">
@@ -184,5 +189,5 @@
                 xyz="-0.0185 0 ${lower_joint_to_tip_distance}"
                 mesh_file="${tip_link_mesh}"
-                material="fingerpro_shell"
+                material="fingerpro_tip"
                 mesh_scale="1."/>
             <xacro:add_inertia

Commit message: Explicitly set mass/inertia of visual link to zero
These links only add visual elements that should not affect the physical
behaviour of the robot.  However, if not specified, pyBullet assumes a
default mass of 1 kg...

File: xacro/pro/fingerpro_macro.xacro (robot description, xacro)
@@ -78,5 +78,5 @@
                 com="0 0.06 0"/>
         </link>
-        <link name="finger_upper_link_motor${suffix}">
+        <link name="finger_upper_link_visuals${suffix}">
             <!-- motor -->
             <visual>
@@ -111,8 +111,12 @@
                 <material name="fingerpro_motor" />
             </visual>
-        </link>
-        <joint name="finger_upper_to_motor_joint${suffix}" type="fixed">
+            <inertial>
+                <mass value="0"/>
+                <inertia ixx="0.0" ixy="0.0" ixz="0.0" iyy="0.0" iyz="0.0" izz="0.0"/>
+            </inertial>
+        </link>
+        <joint name="finger_upper_visuals_joint${suffix}" type="fixed">
             <parent link="finger_upper_link${suffix}"/>
-            <child link="finger_upper_link_motor${suffix}"/>
+            <child link="finger_upper_link_visuals${suffix}"/>
             <origin xyz="0 ${center_offset} 0" />
         </joint>
@@ -131,5 +135,5 @@
                 com="${2 * mesh_x_offset} 0 -0.08"/>
         </link>
-        <link name="finger_middle_link_motor${suffix}">
+        <link name="finger_middle_link_visuals${suffix}">
             <!-- motor -->
             <visual>
@@ -164,8 +168,12 @@
                 <material name="fingerpro_motor" />
             </visual>
-        </link>
-        <joint name="finger_middle_to_motor_joint${suffix}" type="fixed">
+            <inertial>
+                <mass value="0"/>
+                <inertia ixx="0.0" ixy="0.0" ixz="0.0" iyy="0.0" iyz="0.0" izz="0.0"/>
+            </inertial>
+        </link>
+        <joint name="finger_middle_visuals_joint${suffix}" type="fixed">
             <parent link="finger_middle_link${suffix}"/>
-            <child link="finger_middle_link_motor${suffix}"/>
+            <child link="finger_middle_link_visuals${suffix}"/>
         </joint>
         <link name="finger_lower_link${suffix}">

Commit message: Use new, cleaner FingerPro meshes

File: xacro/pro/fingerpro_macro.xacro (robot description, xacro)
@@ -11,11 +11,11 @@
     <!-- Meshes -->
     <xacro:property name="mesh_dir" value="package://robot_properties_fingers/meshes/pro"/>
-    <xacro:property name="center_link_mesh" value="${mesh_dir}/SIM__BL-Finger_Center.stl"/>
-    <xacro:property name="upper_base_mesh" value="${mesh_dir}/SIM__BL-Finger_Base.stl"/>
-    <xacro:property name="upper_link_mesh" value="${mesh_dir}/SIM__BL-Finger_Proximal.stl"/>
-    <xacro:property name="middle_link_mesh" value="${mesh_dir}/SIM__BL-Finger_Intermediate.stl"/>
-    <xacro:property name="lower_link_mesh" value="${mesh_dir}/SIM__BL-Finger_Tip_without_tip.stl"/>
-    <xacro:property name="tip_link_mesh" value="${mesh_dir}/SIM__BL-Finger_Tip_actual_tip.stl"/>
-    <xacro:property name="motor_mesh" value="${mesh_dir}/SIM__BL-Finger_Motor.stl"/>
+    <xacro:property name="center_link_mesh" value="${mesh_dir}/center_axis_sim.stl"/>
+    <xacro:property name="upper_base_mesh" value="${mesh_dir}/detailed/SIM__BL-Finger_Base.stl"/>
+    <xacro:property name="upper_link_mesh" value="${mesh_dir}/prox-sim.stl"/>
+    <xacro:property name="middle_link_mesh" value="${mesh_dir}/int_sim.stl"/>
+    <xacro:property name="lower_link_mesh" value="${mesh_dir}/tip_link_sim.stl"/>
+    <xacro:property name="tip_link_mesh" value="${mesh_dir}/tip_sim.stl"/>
+    <xacro:property name="motor_mesh" value="${mesh_dir}/motor_sim.stl"/>
     <!-- Distance from outer edge of the link to the joint center -->
     <xacro:property name="upper_link_length" value="0.20945" />
@@ -50,4 +50,5 @@
         -->
         <link name="finger_base_link${suffix}">
+            <!--
             <xacro:add_geometry
                 rpy="0 0 0"
@@ -56,15 +57,14 @@
                 material="fingerpro_shell"
                 mesh_scale="1." />
-            <xacro:add_inertia
-                length_x="0.05"
-                length_y="0.05"
-                length_z="0.05"
-                mass="1"
-                com="0 0 0"/>
+            -->
+            <inertial>
+                <mass value="0"/>
+                <inertia ixx="0.0" ixy="0.0" ixz="0.0" iyy="0.0" iyz="0.0" izz="0.0"/>
+            </inertial>
         </link>
         <link name="finger_upper_link${suffix}">
             <xacro:add_geometry
                 rpy="0 0 0"
-                xyz="0 ${center_offset} 0"
+                xyz="0 0 0"
                 mesh_file="${upper_link_mesh}"
                 material="fingerpro_shell"
@@ -122,5 +122,5 @@
         <link name="finger_middle_link${suffix}">
             <xacro:add_geometry
-                rpy="${pi/2} 0 0"
+                rpy="0 0 0"
                 xyz="0 0 0"
                 mesh_file="${middle_link_mesh}"
@@ -178,5 +178,5 @@
         <link name="finger_lower_link${suffix}">
             <xacro:add_geometry
-                rpy="${pi/2} 0 0"
+                rpy="0 0 0"
                 xyz="0 0 0"
                 mesh_file="${lower_link_mesh}"
@@ -193,6 +193,6 @@
         <link name="finger_tip_link${suffix}">
             <xacro:add_geometry
-                rpy="${pi/2} 0 0"
-                xyz="-0.0185 0 ${lower_joint_to_tip_distance}"
+                rpy="0 0 0"
+                xyz="0 0 0"
                 mesh_file="${tip_link_mesh}"
                 material="fingerpro_tip"

File: xacro/pro/trifingerpro.urdf.xacro (robot description, xacro)
@@ -26,10 +26,8 @@
             mesh_scale="1." />
         <!-- add inertial to suppress warning -->
-        <xacro:add_inertia
-            length_x="0.005"
-            length_y="0.005"
-            length_z="0.005"
-            mass="1"
-            com="0 0 0"/>
+        <inertial>
+            <mass value="0"/>
+            <inertia ixx="0.0" ixy="0.0" ixz="0.0" iyy="0.0" iyz="0.0" izz="0.0"/>
+        </inertial>
     </link>
     <joint name="base_to_upper_holder_joint" type="fixed">
