Commit message: Set position of tip and motors to exact values

File: xacro/pro/fingerpro_macro.xacro (robot description, xacro)
@@ -19,13 +19,9 @@
     <xacro:property name="motor_mesh" value="${mesh_dir}/motor_sim.stl"/>
     <!-- Distance from outer edge of the link to the joint center -->
-    <xacro:property name="upper_link_length" value="0.20945" />
     <xacro:property name="middle_dx" value="0.01685" />
-    <xacro:property name="middle_dy" value="0.027" />
-    <xacro:property name="lower_dx" value="0.04922" />
+    <xacro:property name="middle_dy" value="0.05050" />
+    <xacro:property name="lower_dx" value="0.05015" />
     <xacro:property name="lower_dy" value="0.16" />
-    <!-- center offset used to shift the finger by radius of the center piece yet to be added  -->
-    <xacro:property name="center_offset" value="0.0235" />
-    <xacro:property name="mesh_x_offset" value="0.014" />
-    <xacro:property name="lower_joint_to_tip_distance" value="0.1626" />
+    <xacro:property name="lower_joint_to_tip_distance" value="0.160" />
     <material name="fingerpro_shell">
         <!-- colour from image -->
@@ -80,5 +76,5 @@
             <!-- motor -->
             <visual>
-                <origin xyz="0.018 0.141 -0.001" />
+                <origin xyz="0.01569 0.1643 0" />
                 <geometry>
                     <mesh filename="${motor_mesh}"/>
@@ -88,5 +84,5 @@
             <!-- end stop -->
             <visual>
-                <origin xyz="0.015 0.06 0" rpy="0 ${pi/2} 0" />
+                <origin xyz="0.015 0.083 0" rpy="0 ${pi/2} 0" />
                 <geometry>
                     <cylinder length="0.015" radius="0.005"/>
@@ -96,5 +92,5 @@
             <!-- cables -->
             <visual>
-                <origin xyz="-0.008 0.1 0" rpy="${pi/2} 0 0" />
+                <origin xyz="-0.008 0.124 0" rpy="${pi/2} 0 0" />
                 <geometry>
                     <cylinder length="0.12" radius="0.002"/>
@@ -104,5 +100,5 @@
             <!-- opening on lower joint -->
             <visual>
-                <origin xyz="-0.008 0.026 0" rpy="0 ${pi/2} 0" />
+                <origin xyz="-0.0085 0.050 0" rpy="0 ${pi/2} 0" />
                 <geometry>
                     <cylinder length="0.002" radius="0.014"/>
@@ -118,5 +114,5 @@
             <parent link="finger_upper_link${suffix}"/>
             <child link="finger_upper_link_visuals${suffix}"/>
-            <origin xyz="0 ${center_offset} 0" />
+            <origin xyz="0 0 0" />
         </joint>
         <link name="finger_middle_link${suffix}">
@@ -137,5 +133,5 @@
             <!-- motor -->
             <visual>
-                <origin xyz="0.048 0 -0.046" />
+                <origin xyz="0.0488 0 -0.0462" />
                 <geometry>
                     <mesh filename="${motor_mesh}"/>
@@ -145,5 +141,5 @@
             <!-- end stop -->
             <visual>
-                <origin xyz="0.048 0 -0.13" rpy="0 ${pi/2} 0" />
+                <origin xyz="0.0488 0 -0.13" rpy="0 ${pi/2} 0" />
                 <geometry>
                     <cylinder length="0.015" radius="0.005"/>
@@ -208,5 +204,5 @@
             <parent link="finger_lower_link${suffix}"/>
             <child link="finger_tip_link${suffix}"/>
-            <origin xyz="0.0185 0 -${lower_joint_to_tip_distance}"/>
+            <origin xyz="0.019 0 -${lower_joint_to_tip_distance}"/>
         </joint>
         <!-- kinematics -->
@@ -226,5 +222,5 @@
             <limit effort="1000" lower="0.0" upper="1.57" velocity="1000"/>
             <axis xyz="1 0 0"/>
-            <origin rpy="0 0 0" xyz="${middle_dx} ${middle_dy+center_offset} 0"/>
+            <origin rpy="0 0 0" xyz="${middle_dx} ${middle_dy} 0"/>
         </joint>
         <joint name="finger_middle_to_lower_joint${suffix}" type="revolute">

Commit message: Set inertials based on CAD data

File: xacro/pro/fingerpro_macro.xacro (robot description, xacro)
@@ -46,12 +46,4 @@
         -->
         <link name="finger_base_link${suffix}">
-            <!--
-            <xacro:add_geometry
-                rpy="0 0 0"
-                xyz="0 ${upper_link_length+center_offset} 0"
-                mesh_file="${upper_base_mesh}"
-                material="fingerpro_shell"
-                mesh_scale="1." />
-            -->
             <inertial>
                 <mass value="0"/>
@@ -66,10 +58,19 @@
                 material="fingerpro_shell"
                 mesh_scale="1." />
-            <xacro:add_inertia
-                length_x="0.04"
-                length_y="0.14"
-                length_z="0.04"
-                mass="0.26"
-                com="0 0.06 0"/>
+            <inertial>
+                <origin rpy="0 0 0" xyz="0.006 0.122 0.000"/>
+                <mass value="0.26689"/>
+                <inertia
+                    ixx="0.00102362"
+                    ixy="0.00000889"
+                    ixz="-0.00000019"
+                    iyx="0.00000889"
+                    iyy="0.00006450"
+                    iyz="0.00000106"
+                    izx="-0.00000019"
+                    izy="0.00000106"
+                    izz="0.00102225"
+                    />
+            </inertial>
         </link>
         <link name="finger_upper_link_visuals${suffix}">
@@ -123,10 +124,19 @@
                 material="fingerpro_shell"
                 mesh_scale="1." />
-            <xacro:add_inertia
-                length_x="0.04"
-                length_y="0.04"
-                length_z="0.14"
-                mass="0.25"
-                com="${2 * mesh_x_offset} 0 -0.08"/>
+            <inertial>
+                <origin rpy="0 0 0" xyz="0.03935008 -0.00012438 -0.08666705"/>
+                <mass value="0.27163"/>
+                <inertia
+                    ixx="0.00094060"
+                    ixy="-0.00000046"
+                    ixz="-0.00003479"
+                    iyx="-0.00000046"
+                    iyy="0.00094824"
+                    iyz="0.00000164"
+                    izx="-0.00003479"
+                    izy="0.00000164"
+                    izz="0.00007573"
+                    />
+            </inertial>
         </link>
         <link name="finger_middle_link_visuals${suffix}">
@@ -179,10 +189,19 @@
                 material="fingerpro_shell"
                 mesh_scale="1."/>
-            <xacro:add_inertia
-                length_x="0.02"
-                length_y="0.02"
-                length_z="0.14"
-                mass="0.021"
-                com="0 0 -0.06"/>
+            <inertial>
+                <origin rpy="0 0 0" xyz="0.01632700 -0.00001095 -0.04284052"/>
+                <mass value="0.05569"/>
+                <inertia
+                    ixx="0.00013626"
+                    ixy="0.00000000"
+                    ixz="-0.00000662"
+                    iyx="0.00000000"
+                    iyy="0.00013372"
+                    iyz="0.00000004"
+                    izx="-0.00000662"
+                    izy="0.00000004"
+                    izz="0.00000667"
+                    />
+            </inertial>
         </link>
         <!-- fixed link for finger tip -->
@@ -200,4 +219,19 @@
                 com="0 0 0"
                 mass="0.031"/>
+            <inertial>
+                <origin rpy="0 0 0" xyz="-0.00001194 0.00000000 0.01560060"/>
+                <mass value="0.0092"/>
+                <inertia
+                    ixx="0.00000155"
+                    ixy="0.00000000"
+                    ixz="0.00000000"
+                    iyx="0.00000000"
+                    iyy="0.00000155"
+                    iyz="0.00000000"
+                    izx="0.00000000"
+                    izy="0.00000000"
+                    izz="0.00000032"
+                    />
+            </inertial>
         </link>
         <joint name="finger_lower_to_tip_joint${suffix}" type="fixed">
