Commit message: Correct order of fingers

File: xacro/pro/trifingerpro.urdf.xacro (robot description, xacro)
@@ -48,5 +48,4 @@
     <xacro:fingerpro suffix="_120" material="finger_120_material" />
     <xacro:fingerpro suffix="_240" material="finger_240_material" />
-    <!-- <xacro:property name="offset" value="0.04"/> upper_holder to finger offset -->
     <xacro:property name="angle_0" value="${radians(0)}"/>
     <xacro:property name="angle_120" value="${radians(120)}"/>
@@ -55,5 +54,4 @@
         <parent link="upper_holder_link"/>
         <child link="finger_base_link_0"/>
-        <!-- <origin xyz="${center_offset * sin(angle_0)} ${center_offset * cos(angle_0)} 0" rpy="0 0 0"/> -->
         <origin xyz="0 0 0" rpy="0 0 ${angle_0}"/>
     </joint>
@@ -61,12 +59,10 @@
         <parent link="upper_holder_link"/>
         <child link="finger_base_link_120"/>
-        <!-- <origin xyz="${center_offset * sin(angle_120)} ${center_offset * cos(angle_120)} 0" rpy="0 0 -${angle_120}"/> -->
-        <origin xyz="0 0 0" rpy="0 0 ${angle_120}"/>
+        <origin xyz="0 0 0" rpy="0 0 -${angle_120}"/>
     </joint>
     <joint name="holder_to_finger_240" type="fixed">
         <parent link="upper_holder_link"/>
         <child link="finger_base_link_240"/>
-        <!-- <origin xyz="${center_offset * sin(angle_240)} ${center_offset * cos(angle_240)} 0" rpy="0 0 -${angle_240}"/> -->
-        <origin xyz="0 0 0" rpy="0 0 ${angle_240}"/>
+        <origin xyz="0 0 0" rpy="0 0 -${angle_240}"/>
     </joint>
 </robot>

Commit message: Set correct finger height for TriFingerPro
Based on measurement done on a real platform.

File: xacro/pro/trifingerpro.urdf.xacro (robot description, xacro)
@@ -33,5 +33,5 @@
         <parent link="base_link"/>
         <child link="upper_holder_link"/>
-        <origin xyz="0 0 0.34"/>
+        <origin xyz="0 0 0.29"/>
     </joint>
     <material name="finger_0_material">

Commit message: Set realistic colour for TriFingerPro
Do not use the red/green/blue fingers but set the colour to something
that resembles the actual colour of the links.

File: xacro/pro/trifingerpro.urdf.xacro (robot description, xacro)
@@ -4,4 +4,16 @@
     <xacro:include filename="fingerpro_macro.xacro" />
     <xacro:include filename="../macros.xacro" />
+    <material name="finger_0_material">
+        <color rgba="0.6 0.0 0.0 1.0" />
+    </material>
+    <material name="finger_120_material">
+        <color rgba="0.0 0.6 0.0 1.0" />
+    </material>
+    <material name="finger_240_material">
+        <color rgba="0.0 0.0 0.6 1.0" />
+    </material>
+    <material name="real_finger_material">
+        <color rgba="0.83 0.79 0.82 1.0" />
+    </material>
     <!-- Define the global base_link and place all other objects relative to it. -->
     <link name="base_link">
@@ -20,5 +32,5 @@
             xyz="0 0 0"
             mesh_file="${center_link_mesh}"
-            material="finger_material"
+            material="real_finger_material"
             mesh_scale="1." />
         <!-- add inertial to suppress warning -->
@@ -35,17 +47,8 @@
         <origin xyz="0 0 0.29"/>
     </joint>
-    <material name="finger_0_material">
-        <color rgba="0.6 0.0 0.0 1.0" />
-    </material>
-    <material name="finger_120_material">
-        <color rgba="0.0 0.6 0.0 1.0" />
-    </material>
-    <material name="finger_240_material">
-        <color rgba="0.0 0.0 0.6 1.0" />
-    </material>
     <!-- Define the three fingers and place them relative to the upper holder -->
-    <xacro:fingerpro suffix="_0" material="finger_0_material" />
-    <xacro:fingerpro suffix="_120" material="finger_120_material" />
-    <xacro:fingerpro suffix="_240" material="finger_240_material" />
+    <xacro:fingerpro suffix="_0" material="real_finger_material" />
+    <xacro:fingerpro suffix="_120" material="real_finger_material" />
+    <xacro:fingerpro suffix="_240" material="real_finger_material" />
     <xacro:property name="angle_0" value="${radians(0)}"/>
     <xacro:property name="angle_120" value="${radians(120)}"/>

Commit message: TriFingerPro: Use zero-mass inertia for base link
It probably doesn't make a difference technically but looks cleaner this
way.

File: xacro/pro/trifingerpro.urdf.xacro (robot description, xacro)
@@ -10,10 +10,8 @@
     <link name="base_link">
         <!-- add inertial to suppress warning -->
-        <xacro:add_inertia
-            length_x="0.005"
-            length_y="0.005"
-            length_z="0.005"
-            mass="1"
-            com="0 0 0"/>
+        <inertial>
+            <mass value="0"/>
+            <inertia ixx="0.0" ixy="0.0" ixz="0.0" iyy="0.0" iyz="0.0" izz="0.0"/>
+        </inertial>
     </link>
     <!-- Define the upper holder -->
