Commit message: Move files and rename from "new_finger" to "fingerpro"

File: xacro/pro/fingerpro.urdf.xacro (robot description, xacro)
@@ -1,4 +1,4 @@
 <?xml version="1.0" ?>
-<robot name="new_finger" xmlns:xacro="https://ei.is.tuebingen.mpg.de/xacro">
+<robot name="fingerpro" xmlns:xacro="https://ei.is.tuebingen.mpg.de/xacro">
     <!--
     Frames are defined such that they all align with the base frame when all
@@ -8,5 +8,5 @@
     finger tip which should make it easy to place the finger in the world.
     -->
-    <xacro:include filename="new_finger_macro.urdf.xacro" />
+    <xacro:include filename="fingerpro_macro.xacro" />
     <material name="finger_material">
         <color rgba="0.6 0.6 0.6 1.0" />
@@ -16,5 +16,5 @@
     The parameters are automatically set inside the finger_macro file, to accomodate for single finger.
     -->
-    <xacro:new_finger material="finger_material" />
+    <xacro:fingerpro material="finger_material" />
     <!--
     Define the global base link and place the finger relative to it.

File: xacro/pro/fingerpro_macro.xacro (robot description, xacro)
@@ -8,13 +8,13 @@
     finger tip which should make it easy to place the finger in the world.
     -->
-    <xacro:include filename="macros.xacro" />
+    <xacro:include filename="../macros.xacro" />
     <!-- Meshes -->
     <xacro:property name="mesh_file_extension" value="stl"/>
-    <xacro:property name="mesh_dir_new" value="package://robot_properties_fingers/meshes/${mesh_file_extension}/new"/>
-    <xacro:property name="center_link_mesh" value="${mesh_dir_new}/SIM__BL-Finger_Center.${mesh_file_extension}"/>
-    <xacro:property name="upper_base_mesh" value="${mesh_dir_new}/SIM__BL-Finger_Base.${mesh_file_extension}"/>
-    <xacro:property name="upper_link_mesh" value="${mesh_dir_new}/SIM__BL-Finger_Proximal.${mesh_file_extension}"/>
-    <xacro:property name="middle_link_mesh" value="${mesh_dir_new}/SIM__BL-Finger_Intermediate.${mesh_file_extension}"/>
-    <xacro:property name="lower_link_mesh" value="${mesh_dir_new}/SIM__BL-Finger_Tip.${mesh_file_extension}"/>
+    <xacro:property name="mesh_dir" value="package://robot_properties_fingers/meshes/${mesh_file_extension}/pro"/>
+    <xacro:property name="center_link_mesh" value="${mesh_dir}/SIM__BL-Finger_Center.${mesh_file_extension}"/>
+    <xacro:property name="upper_base_mesh" value="${mesh_dir}/SIM__BL-Finger_Base.${mesh_file_extension}"/>
+    <xacro:property name="upper_link_mesh" value="${mesh_dir}/SIM__BL-Finger_Proximal.${mesh_file_extension}"/>
+    <xacro:property name="middle_link_mesh" value="${mesh_dir}/SIM__BL-Finger_Intermediate.${mesh_file_extension}"/>
+    <xacro:property name="lower_link_mesh" value="${mesh_dir}/SIM__BL-Finger_Tip.${mesh_file_extension}"/>
     <!-- Distance from outer edge of the link to the joint center -->
     <xacro:property name="upper_link_length" value="0.20945" />
@@ -31,5 +31,5 @@
     In case of single finger, no "suffix" value is passed.
     -->
-    <xacro:macro name="new_finger" params="material suffix:=''">
+    <xacro:macro name="fingerpro" params="material suffix:=''">
         <!--
         Fixed links for the finger base (parts where the upper link is mounted).

File: xacro/pro/trifingerpro.urdf.xacro (robot description, xacro)
@@ -1,7 +1,7 @@
 <?xml version="1.0" ?>
-<robot name="new_trifinger"
+<robot name="trifingerpro"
     xmlns:xacro="https://ei.is.tuebingen.mpg.de/xacro">
-    <xacro:include filename="new_finger_macro.urdf.xacro" />
-    <xacro:include filename="macros.xacro" />
+    <xacro:include filename="fingerpro_macro.xacro" />
+    <xacro:include filename="../macros.xacro" />
     <!-- Define the global base_link and place all other objects relative to it. -->
     <link name="base_link">
@@ -45,7 +45,7 @@
     </material>
     <!-- Define the three fingers and place them relative to the upper holder -->
-    <xacro:new_finger suffix="_0" material="finger_0_material" />
-    <xacro:new_finger suffix="_120" material="finger_120_material" />
-    <xacro:new_finger suffix="_240" material="finger_240_material" />
+    <xacro:fingerpro suffix="_0" material="finger_0_material" />
+    <xacro:fingerpro suffix="_120" material="finger_120_material" />
+    <xacro:fingerpro suffix="_240" material="finger_240_material" />
     <!-- <xacro:property name="offset" value="0.04"/> upper_holder to finger offset -->
     <xacro:property name="angle_0" value="${radians(0)}"/>

Commit message: Add base_link to single FingerPro
Add a base_link and offset the robot with the same height as in the
TriFingerPro platform.

File: xacro/pro/fingerpro.urdf.xacro (robot description, xacro)
@@ -18,4 +18,11 @@
     Note: Here I've used the center point of the center piece as the origin
     -->
+    <link name="base_link">
+        <!-- add inertial to suppress warning -->
+        <inertial>
+            <mass value="0"/>
+            <inertia ixx="0.0" ixy="0.0" ixz="0.0" iyy="0.0" iyz="0.0" izz="0.0"/>
+        </inertial>
+    </link>
     <link name="center_link">
         <xacro:add_geometry
@@ -32,4 +39,9 @@
             com="0 0 0"/>
     </link>
+    <joint name="base_to_center_joint" type="fixed">
+        <parent link="base_link"/>
+        <child link="center_link"/>
+        <origin xyz="0 0 0.29"/>
+    </joint>
     <joint name="base_to_finger" type="fixed">
         <parent link="center_link"/>
